File: Eagle/f2_OrAnd/AND_OR.brd (EAGLE design)
At the start: 160 x 100 mm, 12 parts, among them IC1 TINY13-20SSU

Commit message: 第一次更新
Parts:
- moved R1 5.27 mm to (94.0, 59.4)
- moved LED1 4.51 mm to (94.0, 63.0), turned to 90 degrees
- moved U$4 0.98 mm to (66.8, 53.5)
Routing:
- net 5V: track 108.0 -> 111.0 mm
- net N$1: track 2.63 -> 1.90 mm
