File: Eagle/f3_Compare/COMPARE.brd (EAGLE design)
At the start: 160 x 100 mm, 9 parts, among them IC2 TINY13-20SSU

Commit message: 第一次更新
Parts:
- moved R1 13.0 mm to (93.9, 65.5)
- moved LED1 10.3 mm to (93.9, 68.8), turned to 90 degrees
Routing:
- net 5V: track 71.0 -> 80.3 mm
- net GND: track 13.8 -> 11.5 mm, vias 10 -> 9
- net N$1: track 2.33 -> 1.70 mm
Changed lines of the file:
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@@
 <?xml version="1.0" encoding="utf-8"?>
 <!DOCTYPE eagle SYSTEM "eagle.dtd">
-<eagle version="7.2.0">
+<eagle version="6.6.0">
 <drawing>
 <settings>
@@
 <pass name="Default">
 <param name="RoutingGrid" value="50mil"/>
-<param name="AutoGrid" value="1"/>
-<param name="Efforts" value="0"/>
-<param name="TopRouterVariant" value="1"/>
 <param name="tpViaShape" value="round"/>
-<param name="PrefDir.1" value="a"/>
+<param name="PrefDir.1" value="|"/>
 <param name="PrefDir.2" value="0"/>
 <param name="PrefDir.3" value="0"/>
@@
 <param name="PrefDir.14" value="0"/>
 <param name="PrefDir.15" value="0"/>
-<param name="PrefDir.16" value="a"/>
+<param name="PrefDir.16" value="-"/>
 <param name="cfVia" value="8"/>
 <param name="cfNonPref" value="5"/>
@@
 <attribute name="NAME" x="73.3425" y="56.261" size="1.27" layer="25" ratio="10" rot="R90"/>
 </element>
-<element name="LED1" library="led" package="SML0603" value="" x="83.566" y="68.834" smashed="yes" rot="R270">
-<attribute name="NAME" x="84.312" y="70.342" size="0.8128" layer="25" rot="R270"/>
-<attribute name="VALUE" x="81.566" y="69.834" size="1.27" layer="27" rot="R270"/>
+<element name="LED1" library="led" package="SML0603" value="" x="93.853" y="68.8086" smashed="yes" rot="R90">
+<attribute name="NAME" x="95.6978" y="67.5292" size="0.8128" layer="25" rot="R90"/>
+<attribute name="VALUE" x="95.853" y="67.8086" size="1.27" layer="27" rot="R90"/>
 </element>
 <element name="C1" library="SparkFun-Capacitors" package="0603-CAP" value="0.1uF" x="71.374" y="61.976" rot="R270">
@@
 <element name="H2" library="HEAD_LOCK" package="HEAD_LOCK" value="HEAD_LOCK" x="59.69" y="49.53"/>
 <element name="H3" library="HEAD_LOCK" package="HEAD_LOCK" value="HEAD_LOCK" x="93.98" y="55.88" rot="R90"/>
-<element name="R1" library="SparkFun-Passives" package="0603-RES" value="" x="81.28" y="68.834" smashed="yes" rot="R90">
-<attribute name="NAME" x="80.264" y="67.945" size="0.8128" layer="25" font="vector" rot="R90"/>
-<attribute name="VALUE" x="82.423" y="67.818" size="0.4064" layer="27" font="vector" rot="R90"/>
+<element name="R1" library="SparkFun-Passives" package="0603-RES" value="" x="93.853" y="65.5066" smashed="yes" rot="R90">
+<attribute name="NAME" x="92.837" y="64.6176" size="0.8128" layer="25" font="vector" rot="R90"/>
+<attribute name="VALUE" x="94.996" y="64.4906" size="0.4064" layer="27" font="vector" rot="R90"/>
 </element>
 <element name="U$1" library="Xmaker_yuhui" package="DIMENSION1" value="DIMENSION1" x="50.8" y="43.18"/>
@@
 <contactref element="R1" pad="1"/>
 <contactref element="H3" pad="3"/>
-<wire x1="81.28" y1="67.984" x2="73.572" y2="67.984" width="0.6096" layer="1"/>
-<wire x1="73.572" y1="67.984" x2="71.374" y2="65.786" width="0.6096" layer="1"/>
-<wire x1="71.374" y1="65.786" x2="71.374" y2="62.826" width="0.6096" layer="1"/>
 <polygon width="0.6096" layer="16">
 <vertex x="46.736" y="75.184"/>
@@
 <via x="67.056" y="58.1406" extent="1-16" drill="0.3048"/>
 <via x="70.0786" y="58.0898" extent="1-16" drill="0.3048"/>
-<via x="77.8002" y="63.373" extent="1-16" drill="0.3048"/>
 <via x="81.534" y="63.2968" extent="1-16" drill="0.3048"/>
 <via x="82.1944" y="55.372" extent="1-16" drill="0.3048"/>
@@
 <via x="74.1172" y="49.1236" extent="1-16" drill="0.3048"/>
 <via x="70.0532" y="49.1236" extent="1-16" drill="0.3048"/>
+<wire x1="93.853" y1="64.6566" x2="93.98" y2="64.6566" width="0.6096" layer="1"/>
+<wire x1="93.98" y1="64.6566" x2="93.98" y2="60.96" width="0.6096" layer="1"/>
+<wire x1="78.095" y1="55.766" x2="85.2548" y2="55.766" width="0.6096" layer="1"/>
+<wire x1="85.2548" y1="55.766" x2="85.6488" y2="55.372" width="0.6096" layer="1"/>
 </signal>
 <signal name="N$1">
 <contactref element="LED1" pad="C"/>
 <contactref element="R1" pad="2"/>
-<wire x1="83.566" y1="69.584" x2="81.38" y2="69.584" width="0.6096" layer="1"/>
-<wire x1="81.38" y1="69.584" x2="81.28" y2="69.684" width="0.6096" layer="1"/>
+<wire x1="93.853" y1="68.0586" x2="93.853" y2="66.3566" width="0.6096" layer="1"/>
 </signal>
 <signal name="5V">
@@
 <wire x1="90.17" y1="58.42" x2="83.566" y2="65.024" width="0.8128" layer="1"/>
 <wire x1="83.566" y1="65.024" x2="83.566" y2="65.3796" width="0.8128" layer="1"/>
-<wire x1="83.566" y1="65.3796" x2="83.566" y2="68.084" width="0.8128" layer="1"/>
 <wire x1="74.295" y1="61.074" x2="74.295" y2="63.7794" width="0.8128" layer="1"/>
 <wire x1="74.295" y1="63.7794" x2="75.946" y2="65.4304" width="0.8128" layer="1"/>
@@
 <wire x1="67.691" y1="68.7324" x2="63.6524" y2="68.7324" width="0.8128" layer="1"/>
 <wire x1="63.6524" y1="68.7324" x2="62.23" y2="67.31" width="0.8128" layer="1"/>
+<wire x1="93.853" y1="69.5586" x2="87.745" y2="69.5586" width="0.6096" layer="1"/>
+<wire x1="87.745" y1="69.5586" x2="83.566" y2="65.3796" width="0.6096" layer="1"/>
 </signal>
 <signal name="SELECT">
