File: Eagle/f4_Delay/DELAY.brd (EAGLE design)
At the start: 160 x 100 mm, 12 parts, among them IC1 TINY13-20SSU

Commit message: 第一次更新
Parts:
- removed U$4: POL_CIRCLE, Xmaker_yuhui:POT_CIRCLE
- added R2: (no value), pot:3RP/1610N
- moved R3 37.0 mm to (84.5, 57.1)
- moved LED2 35.4 mm to (84.4, 60.6), turned to 90 degrees
- moved C2 3.87 mm to (58.7, 51.6), turned to 90 degrees
- moved IC1 2.54 mm to (63.5, 48.3)
Connections:
- net CONTROL: now also R2.2; no longer U$4.P$2
- net GND: now also R2.1; no longer U$4.P$3
- net VCC: now also R2.3; no longer U$4.P$1
Routing:
- net VCC: track 110.7 -> 139.3 mm
- net CONTROL: track 10.6 -> 21.8 mm
- net SELECT: track 25.8 -> 23.2 mm
Other:
- board text added: "GND"
- board text added: "SIG"
- board text added: "VCC"
