File: Eagle/f4_Delay/DELAY.sch (EAGLE design)
At the start: 12 parts, among them IC1 TINY13-20SSU

Commit message: 第一次更新
Parts:
- removed U$4: POL_CIRCLE, Xmaker_yuhui:POL_CIRCLE
- added R2: (no value), pot:3RP/1610N
Connections:
- net CONTROL: now also R2.S; no longer U$4.2
- net GND: now also R2.A; no longer U$4.3
- net VCC: now also R2.E; no longer U$4.1
Changed lines of the file:
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@@
 <part name="H2" library="HEAD_LOCK" deviceset="HEAD_LOCK" device=""/>
 <part name="C2" library="SparkFun-Passives" deviceset="CAP" device="0603-CAP" value="0.1uF"/>
+<part name="R2" library="pot" deviceset="3RP/1610N" device=""/>
 <part name="SUPPLY2" library="supply2" deviceset="GND" device=""/>
 <part name="SUPPLY9" library="supply2" deviceset="GND" device=""/>
@@
 <part name="U$3" library="Xmaker_yuhui" deviceset="OPENHARDWARE" device=""/>
 <part name="SUPPLY1" library="supply2" deviceset="VCC" device=""/>
-<part name="U$4" library="Xmaker_yuhui" deviceset="POL_CIRCLE" device=""/>
 </parts>
 <sheets>
@@
 <instance part="H2" gate="G$1" x="58.42" y="-5.08"/>
 <instance part="C2" gate="G$1" x="-27.94" y="35.56"/>
+<instance part="R2" gate="G$1" x="-15.24" y="-40.64"/>
 <instance part="SUPPLY2" gate="GND" x="-15.24" y="-48.26"/>
 <instance part="SUPPLY9" gate="GND" x="-27.94" y="-10.16"/>
@@
 <instance part="U$3" gate="G$1" x="-48.26" y="-38.1"/>
 <instance part="SUPPLY1" gate="G$1" x="30.48" y="-22.86"/>
-<instance part="U$4" gate="G$1" x="-15.24" y="-40.64"/>
 </instances>
 <busses>
@@
 <nets>
 <net name="GND" class="0">
+<segment>
+<pinref part="R2" gate="G$1" pin="A"/>
+<pinref part="SUPPLY2" gate="GND" pin="GND"/>
+</segment>
 <segment>
 <pinref part="IC1" gate="G$1" pin="GND"/>
@@
 <wire x1="30.48" y1="-48.26" x2="30.48" y2="-53.34" width="0.1524" layer="91"/>
 </segment>
-<segment>
-<pinref part="SUPPLY2" gate="GND" pin="GND"/>
-<pinref part="U$4" gate="G$1" pin="3"/>
-</segment>
 </net>
 <net name="VCC" class="0">
@@
 <pinref part="H1" gate="G$1" pin="2"/>
 <wire x1="-71.12" y1="5.08" x2="-76.2" y2="5.08" width="0.1524" layer="91"/>
+</segment>
+<segment>
+<pinref part="R2" gate="G$1" pin="E"/>
+<pinref part="SUPPLY15" gate="G$1" pin="VCC"/>
 </segment>
 <segment>
@@
 <pinref part="SUPPLY1" gate="G$1" pin="VCC"/>
 </segment>
-<segment>
-<pinref part="SUPPLY15" gate="G$1" pin="VCC"/>
-<pinref part="U$4" gate="G$1" pin="1"/>
-</segment>
 </net>
 <net name="CONTROL" class="0">
@@
 </segment>
 <segment>
+<pinref part="R2" gate="G$1" pin="S"/>
 <wire x1="-10.16" y1="-40.64" x2="2.54" y2="-40.64" width="0.1524" layer="91"/>
-<pinref part="U$4" gate="G$1" pin="2"/>
 </segment>
 </net>
