File: Eagle/f5_Count/COUNT.brd (EAGLE design)
At the start: 160 x 100 mm, 11 parts, among them IC1 TINY13-20SSU

Commit message: 第一次更新
Parts:
- moved R1 9.38 mm to (89.6, 34.8)
- moved S1 8.87 mm to (81.2, 32.3)
- moved R3 4.98 mm to (89.8, 49.1)
- moved LED2 1.07 mm to (91.4, 53.0), turned to 90 degrees
Routing:
- net GND: track 29.9 -> 16.1 mm
- net IN: track 26.9 -> 30.3 mm
- net VCC: track 97.3 -> 94.2 mm
- net N$2: track 1.57 -> 2.96 mm
- net SELECT: track 24.4 -> 25.7 mm
