File: Eagle/i8_InfraredReflective/Grove - Infrared Reflective Sensor.brd (EAGLE design)
At the start: 24.2 x 20 mm, 12 parts, among them U1 002-LMV358

Commit message: 第一次更新
Parts:
- R4: value 10K -> 10k; device rcl:RTRIM3214W -> Discrete:3P-SQUA-6.7X6.4
- moved R4 11.2 mm to (27.5, 35.9)
Routing:
- net VCC: track 25.5 -> 22.1 mm
Changed lines of the file:
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@@
 <?xml version="1.0" encoding="utf-8"?>
 <!DOCTYPE eagle SYSTEM "eagle.dtd">
-<eagle version="7.2.0">
+<eagle version="6.6.0">
 <drawing>
 <settings>
@@
 <pass name="Default">
 <param name="RoutingGrid" value="50mil"/>
-<param name="AutoGrid" value="1"/>
-<param name="Efforts" value="0"/>
-<param name="TopRouterVariant" value="1"/>
 <param name="tpViaShape" value="round"/>
 <param name="PrefDir.1" value="|"/>
@@
 </autorouter>
 <elements>
-<element name="R4" library="rcl" package="RTRIM3214W" value="10K" x="16.383" y="36.068" smashed="yes">
-<attribute name="NAME" x="15.593" y="38.7587" size="0.8128" layer="25" font="vector"/>
-<attribute name="VALUE" x="20.193" y="34.163" size="0.6096" layer="27" rot="R90"/>
-</element>
 <element name="U1" library="ICs" package="SO08" value="002-LMV358" x="9.398" y="31.496" smashed="yes" rot="R180">
 <attribute name="NAME" x="9.525" y="35.56" size="0.8128" layer="25" font="vector"/>
@@
 <element name="H1" library="HEAD_LOCK" package="HEAD_LOCK" value="HEAD_LOCK" x="3.175" y="32.385" rot="R270"/>
 <element name="U$3" library="Xmaker_yuhui" package="XMAKERLOGO2" value="XMAKERLOGO2" x="8.636" y="32.512" rot="MR0"/>
+<element name="R4" library="Discrete" package="3P-SQUA-6.7X6.4" value="10k" x="27.5336" y="35.8902"/>
 </elements>
 <signals>
@@
 <signal name="VCC">
 <contactref element="U1" pad="8"/>
-<contactref element="R4" pad="3"/>
 <contactref element="R3" pad="1"/>
 <contactref element="R1" pad="2"/>
 <contactref element="S1" pad="1"/>
 <wire x1="15.24" y1="30.734" x2="15.24" y2="32.2" width="0.4064" layer="1"/>
-<wire x1="15.24" y1="32.2" x2="17.658" y2="34.618" width="0.4064" layer="1"/>
 <wire x1="11.43" y1="26.162" x2="13.97" y2="26.162" width="0.6096" layer="1"/>
 <wire x1="13.97" y1="26.162" x2="13.97" y2="28.679" width="0.6096" layer="1"/>
@@
 <wire x1="10.922" y1="30.734" x2="11.303" y2="30.353" width="0.6096" layer="1"/>
 <wire x1="11.303" y1="28.8798" x2="11.303" y2="30.353" width="0.6096" layer="1"/>
+<contactref element="R4" pad="3"/>
+<wire x1="15.24" y1="32.2" x2="30.0336" y2="33.3902" width="0" layer="19" extent="1-1"/>
 </signal>
 <signal name="N$1">
-<contactref element="R4" pad="2"/>
 <contactref element="U1" pad="2"/>
 <contactref element="C1" pad="2"/>
@@
 <wire x1="11.43" y1="37.211" x2="12.827" y2="37.211" width="0.6096" layer="1"/>
 <wire x1="12.827" y1="37.211" x2="16.076" y2="37.211" width="0.6096" layer="1"/>
-<wire x1="16.076" y1="37.211" x2="16.383" y2="37.518" width="0.6096" layer="1"/>
+<contactref element="R4" pad="2"/>
+<wire x1="27.5336" y1="38.3902" x2="10.033" y2="34.1122" width="0" layer="19" extent="1-1"/>
 </signal>
 <signal name="GND">
 <contactref element="U1" pad="4"/>
-<contactref element="R4" pad="1"/>
 <contactref element="S1" pad="3"/>
 <contactref element="R2" pad="1"/>
@@
 </polygon>
 <contactref element="H1" pad="3"/>
+<contactref element="R4" pad="1"/>
+<wire x1="13.99" y1="31.499" x2="25.0336" y2="33.3902" width="0" layer="19" extent="1-1"/>
+<wire x1="12.827" y1="35.687" x2="13.99" y2="31.499" width="0" layer="19" extent="1-1"/>
+<wire x1="7.493" y1="34.1122" x2="12.827" y2="35.687" width="0" layer="19" extent="1-1"/>
+<wire x1="16.51" y1="24.638" x2="13.99" y2="31.499" width="0" layer="19" extent="1-1"/>
+<wire x1="3.175" y1="27.305" x2="7.493" y2="34.1122" width="0" layer="19" extent="1-1"/>
 </signal>
 <signal name="N$12">
