File: Eagle/arduino_miniuno.brd (EAGLE design)
At the start: 160 x 100 mm, 40 parts, among them J3 1X7P-2.54-2.54-6.0-90D-1, Q1 S8550, Q2 S8550, T1 FDN340P, U1 CH340T, U2 NCP1117ST50T3G, U3 LP2985-33DBVR, U5 LMV358IDGKR, X1 12MHz, X2 USB-B_TH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

Commit message: miniuno
Parts:
- moved U$3 260.9 mm to (92.7, 48.3), turned to 270 degrees
- moved PCB2 216.4 mm to (52.1, 30.5)
- moved X2 106.8 mm to (63.5, 68.6), turned to 270 degrees
Connections:
- new net A6: U$3.A6
- new net A7: U$3.A7
- net A4: now also U$3.A4
- net A5: now also U$3.A5
