File: Eagle/arduino_miniuno.sch (EAGLE design)
At the start: 40 parts, among them J3 1X7P-2.54-2.54-6.0-90D-1, Q1 S8550, Q2 S8550, T1 FDN340P, U1 CH340T, U2 NCP1117ST50T3G, U3 LP2985-33DBVR, U5 LMV358IDGKR, X1 12MHz, X2 USB-B_TH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

Commit message: miniuno
Connections:
- new net A6: U$3.A6
- new net A7: U$3.A7
- net A4: now also U$3.A4
- net A5: now also U$3.A5
Changed lines of the file:
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@@
 <label x="335.28" y="-68.58" size="1.778" layer="95" rot="R90"/>
+</segment>
+<segment>
+<pinref part="U$3" gate="G$1" pin="A5"/>
+<wire x1="332.74" y1="20.32" x2="337.82" y2="20.32" width="0.1524" layer="91"/>
+<label x="335.28" y="20.32" size="1.778" layer="95"/>
 </segment>
 </net>
@@
 <wire x1="332.74" y1="-60.96" x2="332.74" y2="-66.04" width="0.1524" layer="91"/>
 <label x="332.74" y="-68.58" size="1.778" layer="95" rot="R90"/>
+</segment>
+<segment>
+<pinref part="U$3" gate="G$1" pin="A4"/>
+<wire x1="332.74" y1="15.24" x2="337.82" y2="15.24" width="0.1524" layer="91"/>
+<label x="335.28" y="15.24" size="1.778" layer="95"/>
 </segment>
 </net>
@@
 </segment>
 </net>
+<net name="A7" class="0">
+<segment>
+<pinref part="U$3" gate="G$1" pin="A7"/>
+<wire x1="332.74" y1="33.02" x2="337.82" y2="33.02" width="0.1524" layer="91"/>
+<label x="335.28" y="33.02" size="1.778" layer="95"/>
+</segment>
+</net>
+<net name="A6" class="0">
+<segment>
+<pinref part="U$3" gate="G$1" pin="A6"/>
+<wire x1="332.74" y1="27.94" x2="337.82" y2="27.94" width="0.1524" layer="91"/>
+<label x="335.28" y="27.94" size="1.778" layer="95"/>
+</segment>
+</net>
