File: Eagle/o1_LED/Eagle_LED.brd (EAGLE design)
At the start: 20 x 24.2 mm, 11 parts, among them Q1 S9013

Commit message: miniuno
Parts:
- removed H1: HEAD_LOCK, HEAD_LOCK:HEAD_LOCK
- removed Q1: S9013, Discrete:SOT23
- removed R2: 1K, Discrete:3P-SQUA-6.7X6.4
- removed R3: 220, Discrete:0603
- removed R4: 1K, Discrete:0603
- removed R5: 100K, Discrete:0603
- added HEAD_LOCK1: HEAD_LOCK, Xmaker_yuhuilbr:HEAD_LOCK
- moved R1 13.8 mm to (-1.02, 8.38)
Connections:
- removed net N$2: D1.-, Q1.3
- removed net N$3: D1.+, R3.2
- removed net N$4: Q1.1, R4.2, R5.2
- net GND: now also D1.-, HEAD_LOCK1.3; no longer H1.3, Q1.2, R5.1
- net N$1: now also D1.+; no longer R2.2, R2.3, R3.1
- net SIG: now also HEAD_LOCK1.1, R1.1; no longer H1.1, R4.1
- net VCC: now also HEAD_LOCK1.2; no longer H1.2, R1.1, R2.1
Routing:
- net N$1: track 16.5 -> 0.00 mm
- net VCC: track 14.3 -> 0.00 mm
- net GND: track 12.8 -> 0.00 mm, vias 1 -> 0
- net N$4: track 6.02 -> 0.00 mm
- net N$3: track 5.71 -> 0.00 mm
- net N$2: track 3.99 -> 0.00 mm
- net SIG: track 4.02 -> 0.72 mm
Changed lines of the file:
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@@
 </autorouter>
 <elements>
-<element name="R1" library="Discrete" package="0603" value="1K" x="11.684" y="13.716" rot="R180"/>
 <element name="D1" library="Discrete" package="LED-2P-2.54-6MM" value="" x="4.318" y="18.796" rot="R180"/>
-<element name="R2" library="Discrete" package="3P-SQUA-6.7X6.4" value="1K" x="11.43" y="21.082" rot="R90"/>
-<element name="R3" library="Discrete" package="0603" value="220" x="7.874" y="13.716" rot="R180"/>
-<element name="Q1" library="Discrete" package="SOT23" value="S9013" x="0.762" y="14.732"/>
-<element name="R4" library="Discrete" package="0603" value="1K" x="-1.016" y="8.382" rot="R180"/>
-<element name="R5" library="Discrete" package="0603" value="100K" x="-1.016" y="10.668" rot="R180"/>
-<element name="H1" library="HEAD_LOCK" package="HEAD_LOCK" value="HEAD_LOCK" x="3.556" y="8.89"/>
+<element name="R1" library="Discrete" package="0603" value="1K" x="-1.016" y="8.382" rot="R180"/>
 <element name="U$4" library="switch-tact" package="XMAKERLOGO" value="XMAKERLOGO" x="-3.048" y="7.62"/>
 <element name="U$2" library="Xmaker_yuhui" package="DIMENSION" value="DIMENSION" x="6.35" y="11.43"/>
 <element name="U$6" library="SparkFun-Aesthetics" package="OSHW-LOGO-S" value="" x="13.589" y="9.398"/>
+<element name="HEAD_LOCK1" library="Xmaker_yuhuilbr" package="HEAD_LOCK" value="HEAD_LOCK" x="3.048" y="-2.032"/>
 </elements>
 <signals>
-<signal name="N$1">
-<contactref element="R1" pad="2"/>
-<contactref element="R2" pad="2"/>
-<contactref element="R3" pad="1"/>
-<contactref element="R2" pad="3"/>
-<wire x1="13.93" y1="23.582" x2="11.43" y2="23.582" width="0.4064" layer="16"/>
-<wire x1="11.43" y1="23.582" x2="8.93" y2="21.082" width="0.4064" layer="16"/>
-<wire x1="10.922" y1="13.716" x2="8.636" y2="13.716" width="0.4064" layer="1"/>
-<wire x1="10.922" y1="13.716" x2="8.93" y2="15.708" width="0.4064" layer="1"/>
-<wire x1="8.93" y1="15.708" x2="8.93" y2="21.082" width="0.4064" layer="1"/>
-</signal>
 <signal name="GND">
-<contactref element="H1" pad="3"/>
-<contactref element="Q1" pad="2"/>
-<contactref element="R5" pad="1"/>
-<wire x1="1.651" y1="13.716" x2="-0.254" y2="11.811" width="0.4064" layer="1"/>
-<wire x1="-0.254" y1="11.811" x2="-0.254" y2="10.668" width="0.4064" layer="1"/>
-<wire x1="8.636" y1="8.89" x2="4.318" y2="13.208" width="0.4064" layer="16"/>
-<via x="4.318" y="13.208" extent="1-16" drill="0.6" shape="square"/>
-<wire x1="4.318" y1="13.208" x2="2.159" y2="13.208" width="0.4064" layer="1"/>
-<wire x1="2.159" y1="13.208" x2="1.651" y2="13.716" width="0.4064" layer="1"/>
 <polygon width="0.4064" layer="1">
 <vertex x="-3.81" y="26.416"/>
@@
 <vertex x="-3.81" y="4.572"/>
 </polygon>
+<contactref element="D1" pad="-"/>
+<contactref element="HEAD_LOCK1" pad="3"/>
+<wire x1="3.0734" y1="-4.6228" x2="3.0482" y2="18.796" width="0" layer="19" extent="1-1"/>
+</signal>
+<signal name="SIG">
+<contactref element="R1" pad="1"/>
+<wire x1="-0.254" y1="8.382" x2="0.254" y2="8.89" width="0.4064" layer="1"/>
+<contactref element="HEAD_LOCK1" pad="1"/>
+<wire x1="3.0734" y1="0.4572" x2="-0.254" y2="8.382" width="0" layer="19" extent="1-1"/>
+</signal>
+<signal name="N$1">
+<contactref element="R1" pad="2"/>
+<contactref element="D1" pad="+"/>
+<wire x1="-1.778" y1="8.382" x2="5.5878" y2="18.796" width="0" layer="19" extent="1-1"/>
 </signal>
 <signal name="VCC">
-<contactref element="H1" pad="2"/>
-<contactref element="R2" pad="1"/>
-<contactref element="R1" pad="1"/>
-<wire x1="13.93" y1="18.582" x2="12.446" y2="17.098" width="0.4064" layer="1"/>
-<wire x1="12.446" y1="17.098" x2="12.446" y2="13.716" width="0.4064" layer="1"/>
-<wire x1="12.446" y1="13.716" x2="9.906" y2="11.176" width="0.4064" layer="1"/>
-<wire x1="9.906" y1="11.176" x2="7.62" y2="11.176" width="0.4064" layer="1"/>
-<wire x1="7.62" y1="11.176" x2="6.096" y2="9.652" width="0.4064" layer="1"/>
-<wire x1="6.096" y1="9.652" x2="6.096" y2="8.89" width="0.4064" layer="1"/>
-</signal>
-<signal name="N$3">
-<contactref element="R3" pad="2"/>
-<contactref element="D1" pad="+"/>
-<wire x1="7.112" y1="13.716" x2="5.5878" y2="15.2402" width="0.4064" layer="1"/>
-<wire x1="5.5878" y1="15.2402" x2="5.5878" y2="18.796" width="0.4064" layer="1"/>
-</signal>
-<signal name="SIG">
-<contactref element="R4" pad="1"/>
-<contactref element="H1" pad="1"/>
-<wire x1="-0.254" y1="8.382" x2="0.254" y2="8.89" width="0.4064" layer="1"/>
-<wire x1="0.254" y1="8.89" x2="3.556" y2="8.89" width="0.4064" layer="1"/>
-</signal>
-<signal name="N$2">
-<contactref element="Q1" pad="3"/>
-<contactref element="D1" pad="-"/>
-<wire x1="3.0482" y1="18.796" x2="0.762" y2="16.5098" width="0.4064" layer="1"/>
-<wire x1="0.762" y1="16.5098" x2="0.762" y2="15.748" width="0.4064" layer="1"/>
-</signal>
-<signal name="N$4">
-<contactref element="Q1" pad="1"/>
-<contactref element="R4" pad="2"/>
-<contactref element="R5" pad="2"/>
-<wire x1="-0.127" y1="13.716" x2="-1.778" y2="12.065" width="0.4064" layer="1"/>
-<wire x1="-1.778" y1="12.065" x2="-1.778" y2="10.668" width="0.4064" layer="1"/>
-<wire x1="-1.778" y1="10.668" x2="-1.778" y2="8.382" width="0.4064" layer="1"/>
+<contactref element="HEAD_LOCK1" pad="2"/>
 </signal>
 </signals>
