File: Eagle/o4_PWM/PWM.sch (EAGLE design)
At the start: 10 parts, among them IC1 TINY13-20SSU

Commit message: 第一次更新
Parts:
- removed H1, H2: HEAD_LOCK, HEAD_LOCK:HEAD_LOCK
- added HEAD_LOCK1, HEAD_LOCK2: HEAD_LOCK, Xmaker_yuhui:HEAD_LOCK
- U$2: value XMAKERLOGO2 -> XMAKERLOGO_5MM_TOP; device Xmaker_yuhui:XMAKERLOGO2 -> Xmaker_yuhui:XMAKERLOGO_5MM_TOP
- U$4: value OPENHARDWARE -> OPENHARDWARE_5MM_TOP; device Xmaker_yuhui:OPENHARDWARE -> Xmaker_yuhui:OPENHARDWARE_5MM_TOP
Connections:
- net ADC: now also HEAD_LOCK1.1; no longer H1.1
- net GND: now also HEAD_LOCK1.3, HEAD_LOCK2.3; no longer H1.3, H2.3
- net PWM: now also HEAD_LOCK2.1; no longer H2.1
- net VCC: now also HEAD_LOCK1.2, HEAD_LOCK2.2; no longer H1.2, H2.2
Changed lines of the file:
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@@
 <?xml version="1.0" encoding="utf-8"?>
 <!DOCTYPE eagle SYSTEM "eagle.dtd">
-<eagle version="7.2.0">
+<eagle version="6.6.0">
 <drawing>
 <settings>
@@
 <parts>
 <part name="IC1" library="atmel" deviceset="TINY13" device="SSU" technology="-20"/>
-<part name="H1" library="HEAD_LOCK" deviceset="HEAD_LOCK" device=""/>
-<part name="H2" library="HEAD_LOCK" deviceset="HEAD_LOCK" device=""/>
 <part name="C1" library="SparkFun-Passives" deviceset="CAP" device="0603-CAP" value="0.1uF"/>
 <part name="SUPPLY1" library="supply2" deviceset="GND" device=""/>
@@
 <part name="SUPPLY13" library="supply2" deviceset="VCC" device=""/>
 <part name="LED1" library="eagle-ltspice" deviceset="LED_E" device="SML0603"/>
-<part name="U$2" library="Xmaker_yuhui" deviceset="XMAKERLOGO2" device=""/>
 <part name="U$3" library="Xmaker_yuhui" deviceset="DIMENSION1" device=""/>
-<part name="U$4" library="Xmaker_yuhui" deviceset="OPENHARDWARE" device=""/>
 <part name="U$1" library="Xmaker_yuhui" deviceset="POL_CIRCLE" device=""/>
+<part name="HEAD_LOCK1" library="Xmaker_yuhui" deviceset="HEAD_LOCK" device=""/>
+<part name="HEAD_LOCK2" library="Xmaker_yuhui" deviceset="HEAD_LOCK" device=""/>
+<part name="U$2" library="Xmaker_yuhui" deviceset="XMAKERLOGO_5MM_TOP" device=""/>
+<part name="U$4" library="Xmaker_yuhui" deviceset="OPENHARDWARE_5MM_TOP" device=""/>
 </parts>
 <sheets>
@@
 <instances>
 <instance part="IC1" gate="G$1" x="68.58" y="50.8"/>
-<instance part="H1" gate="G$1" x="-12.7" y="76.2"/>
-<instance part="H2" gate="G$1" x="-12.7" y="27.94"/>
 <instance part="C1" gate="G$1" x="40.64" y="88.9"/>
 <instance part="SUPPLY1" gate="GND" x="-7.62" y="48.26"/>
@@
 <instance part="SUPPLY13" gate="G$1" x="63.5" y="106.68"/>
 <instance part="LED1" gate="G$1" x="63.5" y="99.06"/>
-<instance part="U$2" gate="G$1" x="38.1" y="27.94"/>
 <instance part="U$3" gate="G$1" x="63.5" y="25.4"/>
-<instance part="U$4" gate="G$1" x="38.1" y="15.24"/>
 <instance part="U$1" gate="G$1" x="-7.62" y="55.88"/>
+<instance part="HEAD_LOCK1" gate="G$1" x="-7.62" y="83.82"/>
+<instance part="HEAD_LOCK2" gate="G$1" x="-7.62" y="35.56"/>
+<instance part="U$2" gate="G$1" x="40.64" y="27.94"/>
+<instance part="U$4" gate="G$1" x="22.86" y="25.4"/>
 </instances>
 <busses>
@@
 </segment>
 <segment>
-<pinref part="H2" gate="G$1" pin="3"/>
 <pinref part="SUPPLY3" gate="GND" pin="GND"/>
 <wire x1="0" y1="33.02" x2="5.08" y2="33.02" width="0.1524" layer="91"/>
 <wire x1="5.08" y1="33.02" x2="5.08" y2="30.48" width="0.1524" layer="91"/>
-</segment>
-<segment>
-<pinref part="H1" gate="G$1" pin="3"/>
+<pinref part="HEAD_LOCK2" gate="G$1" pin="3"/>
+</segment>
+<segment>
 <pinref part="SUPPLY4" gate="GND" pin="GND"/>
 <wire x1="0" y1="81.28" x2="5.08" y2="81.28" width="0.1524" layer="91"/>
 <wire x1="5.08" y1="81.28" x2="5.08" y2="78.74" width="0.1524" layer="91"/>
+<pinref part="HEAD_LOCK1" gate="G$1" pin="3"/>
 </segment>
 <segment>
@@
 <segment>
 <pinref part="SUPPLY6" gate="G$1" pin="VCC"/>
-<pinref part="H2" gate="G$1" pin="2"/>
 <wire x1="5.08" y1="35.56" x2="0" y2="35.56" width="0.1524" layer="91"/>
+<pinref part="HEAD_LOCK2" gate="G$1" pin="2"/>
 </segment>
 <segment>
 <pinref part="SUPPLY5" gate="G$1" pin="VCC"/>
-<pinref part="H1" gate="G$1" pin="2"/>
 <wire x1="5.08" y1="83.82" x2="0" y2="83.82" width="0.1524" layer="91"/>
+<pinref part="HEAD_LOCK1" gate="G$1" pin="2"/>
 </segment>
 <segment>
@@
 </segment>
 <segment>
-<pinref part="H2" gate="G$1" pin="1"/>
 <wire x1="0" y1="38.1" x2="12.7" y2="38.1" width="0.1524" layer="91"/>
 <label x="5.08" y="38.1" size="1.778" layer="95"/>
+<pinref part="HEAD_LOCK2" gate="G$1" pin="1"/>
 </segment>
 </net>
@@
 </segment>
 <segment>
-<pinref part="H1" gate="G$1" pin="1"/>
 <wire x1="0" y1="86.36" x2="10.16" y2="86.36" width="0.1524" layer="91"/>
 <label x="2.54" y="86.36" size="1.778" layer="95"/>
+<pinref part="HEAD_LOCK1" gate="G$1" pin="1"/>
 </segment>
 </net>

Commit message: 12.15
Parts:
- removed U$1: POL_CIRCLE, Xmaker_yuhui:POL_CIRCLE
- added U$5: POL_CIRCLE, Xmaker:POL_CIRCLE
- HEAD_LOCK1, HEAD_LOCK2: device Xmaker_yuhui:HEAD_LOCK -> Xmaker:HEAD_LOCK
Connections:
- net CONTROL: now also U$5.2; no longer U$1.2
- net GND: now also U$5.3; no longer U$1.3
- net VCC: now also U$5.1; no longer U$1.1
Changed lines of the file:
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@@
 <part name="LED1" library="eagle-ltspice" deviceset="LED_E" device="SML0603"/>
 <part name="U$3" library="Xmaker_yuhui" deviceset="DIMENSION1" device=""/>
-<part name="U$1" library="Xmaker_yuhui" deviceset="POL_CIRCLE" device=""/>
-<part name="HEAD_LOCK1" library="Xmaker_yuhui" deviceset="HEAD_LOCK" device=""/>
-<part name="HEAD_LOCK2" library="Xmaker_yuhui" deviceset="HEAD_LOCK" device=""/>
 <part name="U$2" library="Xmaker_yuhui" deviceset="XMAKERLOGO_5MM_TOP" device=""/>
 <part name="U$4" library="Xmaker_yuhui" deviceset="OPENHARDWARE_5MM_TOP" device=""/>
+<part name="U$5" library="Xmaker" deviceset="POL_CIRCLE" device=""/>
+<part name="HEAD_LOCK1" library="Xmaker" deviceset="HEAD_LOCK" device=""/>
+<part name="HEAD_LOCK2" library="Xmaker" deviceset="HEAD_LOCK" device=""/>
 </parts>
 <sheets>
@@
 <instance part="LED1" gate="G$1" x="63.5" y="99.06"/>
 <instance part="U$3" gate="G$1" x="63.5" y="25.4"/>
-<instance part="U$1" gate="G$1" x="-7.62" y="55.88"/>
+<instance part="U$2" gate="G$1" x="40.64" y="27.94"/>
+<instance part="U$4" gate="G$1" x="22.86" y="25.4"/>
+<instance part="U$5" gate="G$1" x="-7.62" y="55.88"/>
 <instance part="HEAD_LOCK1" gate="G$1" x="-7.62" y="83.82"/>
 <instance part="HEAD_LOCK2" gate="G$1" x="-7.62" y="35.56"/>
-<instance part="U$2" gate="G$1" x="40.64" y="27.94"/>
-<instance part="U$4" gate="G$1" x="22.86" y="25.4"/>
 </instances>
 <busses>
@@
 <segment>
 <pinref part="SUPPLY1" gate="GND" pin="GND"/>
-<pinref part="U$1" gate="G$1" pin="3"/>
+<pinref part="U$5" gate="G$1" pin="3"/>
 </segment>
 </net>
@@
 <segment>
 <pinref part="SUPPLY8" gate="G$1" pin="VCC"/>
-<pinref part="U$1" gate="G$1" pin="1"/>
+<pinref part="U$5" gate="G$1" pin="1"/>
 </segment>
 </net>
@@
 <segment>
 <wire x1="-2.54" y1="55.88" x2="10.16" y2="55.88" width="0.1524" layer="91"/>
-<pinref part="U$1" gate="G$1" pin="2"/>
+<pinref part="U$5" gate="G$1" pin="2"/>
 </segment>
 </net>
