File: Eagle/arduino_miniuno/arduino_miniuno.brd (EAGLE design)
At the start: 160 x 100 mm, 40 parts, among them J3 1X7P-2.54-2.54-6.0-90D-1, Q1 S8550, Q2 S8550, T1 FDN340P, U1 CH340T, U2 NCP1117ST50T3G, U3 LP2985-33DBVR, U5 LMV358IDGKR, X1 12MHz, X2 USB-B_TH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

Commit message: 12.15
Parts:
- removed J3: 1X7P-2.54-2.54-6.0-90D-1, Connector :7P-2.54-65/35MIL
- moved U1 140.6 mm to (84.8, 67.3)
- moved U2 115.8 mm to (40.6, 35.3)
- moved PC2 113.0 mm to (50.5, 20.8)
- moved PC1 110.2 mm to (38.9, 19.8)
- moved C2 92.0 mm to (27.9, 21.6)
- moved D3 86.8 mm to (24.9, 28.2)
- moved L 64.6 mm to (22.1, 11.4)
- moved U3 62.9 mm to (18.5, 17.3)
- moved T1 59.3 mm to (7.11, 19.8)
- moved C1 54.9 mm to (50.0, 6.10)
- moved RN1 52.0 mm to (28.7, 8.38)
- moved RN2 51.1 mm to (39.9, 8.13)
- moved U5 47.6 mm to (10.4, 9.65)
- moved C3 44.2 mm to (45.2, 8.89)
Connections:
- removed net RTS: J3.7, U1.16
- net 5V: no longer J3.4
- net CTS: no longer J3.5
- net DTR: no longer J3.1
- net GND: no longer J3.6
- net RX: no longer J3.2
- net TX: no longer J3.3
