File: Eagle/arduino_miniuno/arduino_miniuno.sch (EAGLE design)
At the start: 40 parts, among them J3 1X7P-2.54-2.54-6.0-90D-1, Q1 S8550, Q2 S8550, T1 FDN340P, U1 CH340T, U2 NCP1117ST50T3G, U3 LP2985-33DBVR, U5 LMV358IDGKR, X1 12MHz, X2 USB-B_TH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

Commit message: 12.15
Parts:
- removed J3: 1X7P-2.54-2.54-6.0-90D-1, Connector :HEADER-7P
Connections:
- removed net RTS: J3.7, U1.RTS#
- net 5V: no longer J3.4
- net CTS: no longer J3.5
- net DTR: no longer J3.1
- net GND: no longer J3.6
- net RX: no longer J3.2
- net TX: no longer J3.3
Changed lines of the file:
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@@
 <part name="U$10" library="Power or GND " deviceset="GND_POWER" device=""/>
 <part name="U$4" library="Power or GND " deviceset="GND_POWER" device=""/>
-<part name="J3" library="Connector " deviceset="HEADER-7P" device="" value="1X7P-2.54-2.54-6.0-90D-1"/>
 <part name="C2" library="SmartPrj" deviceset="C-EU" device="0603-RND" value="100n"/>
 <part name="GND7" library="supply1" deviceset="GND" device=""/>
@@
 <instance part="U$10" gate="G$1" x="142.24" y="22.86" rot="R270"/>
 <instance part="U$4" gate="G$1" x="132.08" y="31.75"/>
-<instance part="J3" gate="G$1" x="203.2" y="11.43" rot="R270"/>
 <instance part="C2" gate="G$1" x="109.22" y="-45.72" smashed="yes" rot="R180">
 <attribute name="NAME" x="101.6" y="-43.18" size="1.778" layer="95"/>
@@
 </segment>
 <segment>
-<wire x1="198.12" y1="19.05" x2="198.12" y2="25.4" width="0.1524" layer="91"/>
-<label x="198.12" y="24.13" size="1.27" layer="95" ratio="10" rot="R270"/>
-<pinref part="J3" gate="G$1" pin="6"/>
-</segment>
-<segment>
 <pinref part="U$5" gate="G$1" pin="GND"/>
 <pinref part="C5" gate="C" pin="1"/>
@@
 <junction x="196.85" y="-15.24"/>
 </segment>
-<segment>
-<wire x1="203.2" y1="19.05" x2="203.2" y2="25.4" width="0.1524" layer="91"/>
-<label x="203.2" y="24.13" size="1.27" layer="95" ratio="10" rot="R270"/>
-<pinref part="J3" gate="G$1" pin="4"/>
-</segment>
 </net>
 <net name="V3" class="0">
@@
 <net name="DTR" class="0">
 <segment>
-<wire x1="210.82" y1="19.05" x2="210.82" y2="25.4" width="0.1524" layer="91"/>
-<label x="210.82" y="24.13" size="1.27" layer="95" ratio="10" rot="R270"/>
-<pinref part="J3" gate="G$1" pin="1"/>
-</segment>
-<segment>
 <pinref part="U1" gate="G$1" pin="DTR#"/>
 <wire x1="177.8" y1="20.32" x2="182.88" y2="20.32" width="0.1524" layer="91"/>
@@
 <pinref part="D1" gate="G$1" pin="2"/>
 <wire x1="210.82" y1="33.02" x2="210.82" y2="34.29" width="0.1524" layer="91"/>
-<pinref part="J3" gate="G$1" pin="2"/>
 </segment>
 <segment>
@@
 <wire x1="205.74" y1="33.02" x2="203.2" y2="33.02" width="0.1524" layer="91"/>
 <wire x1="203.2" y1="33.02" x2="203.2" y2="34.29" width="0.1524" layer="91"/>
-<pinref part="J3" gate="G$1" pin="3"/>
 </segment>
 <segment>
@@
 <net name="CTS" class="0">
 <segment>
-<wire x1="200.66" y1="19.05" x2="200.66" y2="25.4" width="0.1524" layer="91"/>
-<label x="200.66" y="24.13" size="1.27" layer="95" ratio="10" rot="R270"/>
-<pinref part="J3" gate="G$1" pin="5"/>
-</segment>
-<segment>
 <pinref part="U1" gate="G$1" pin="CTS#"/>
 <wire x1="177.8" y1="10.16" x2="182.88" y2="10.16" width="0.1524" layer="91"/>
@@
 <pinref part="R5" gate="R" pin="2"/>
 <wire x1="196.85" y1="-39.37" x2="196.85" y2="-30.48" width="0.1524" layer="91"/>
-</segment>
-</net>
-<net name="RTS" class="0">
-<segment>
-<pinref part="U1" gate="G$1" pin="RTS#"/>
-<wire x1="181.61" y1="22.86" x2="177.8" y2="22.86" width="0.1524" layer="91"/>
-<label x="179.07" y="22.86" size="1.27" layer="95" ratio="10"/>
-</segment>
-<segment>
-<pinref part="J3" gate="G$1" pin="7"/>
-<wire x1="195.58" y1="19.05" x2="195.58" y2="25.4" width="0.1524" layer="91"/>
-<label x="195.58" y="24.13" size="1.27" layer="95" ratio="10" rot="R270"/>
 </segment>
 </net>
@@
 <segment>
 <wire x1="307.34" y1="-17.78" x2="307.34" y2="-12.7" width="0.1524" layer="91"/>
-<label x="307.34" y="-15.24" size="1.778" layer="95" rot="R90"/>
+<label x="307.34" y="-12.7" size="1.778" layer="95" rot="R90"/>
 <pinref part="PCB1" gate="G$1" pin="~9"/>
 </segment>
