File: Eagle/i1_Button/Eagle_Button.brd (EAGLE design)
At the start: 7 parts, among them SW2 BTN

Commit message: chuange touch
Parts:
- moved SW2 1.00 mm to (9.95, 14.3)
Routing:
- net D1: track 16.3 -> 17.3 mm
- net VCC: track 8.29 -> 9.07 mm
Other:
- board text removed: "Button"
Changed lines of the file:
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@@
 <setting verticaltext="up"/>
 </settings>
-<grid distance="1" unitdist="mil" unit="mil" style="lines" multiple="1" display="yes" altdistance="20" altunitdist="mil" altunit="mil"/>
+<grid distance="1" unitdist="mm" unit="mm" style="lines" multiple="1" display="yes" altdistance="20" altunitdist="mil" altunit="mil"/>
 <layers>
 <layer number="1" name="Top" color="4" fill="1" visible="yes" active="yes"/>
@@
 <board>
 <plain>
-<text x="17.288" y="7.668" size="1.27" layer="22" ratio="3" rot="MR270">Button</text>
 </plain>
 <attributes>
@@
 <attribute name="VALUE" x="3.7625" y="3.604" size="0.635" layer="27" ratio="10" rot="R90"/>
 </element>
-<element name="SW2" library="Switch_jumpers" package="BTN_8X8" value="BTN" x="9.9474" y="13.256" smashed="yes" rot="R180">
-<attribute name="NAME" x="14.289" y="14.2338" size="0.8128" layer="25" font="vector" rot="R270"/>
-<attribute name="VALUE" x="12.4574" y="14.066" size="0.8128" layer="27" rot="R180"/>
+<element name="SW2" library="Switch_jumpers" package="BTN_8X8" value="BTN" x="9.9474" y="14.256" smashed="yes" rot="R180">
+<attribute name="NAME" x="14.289" y="15.2338" size="0.8128" layer="25" font="vector" rot="R270"/>
+<attribute name="VALUE" x="12.4574" y="15.066" size="0.8128" layer="27" rot="R180"/>
 </element>
 <element name="H1" library="Xmaker" package="HEAD_LOCK_3PIN_2" value="HEAD_LOCK_3PIN_2" x="9.9728" y="4.7978" smashed="yes" rot="R90">
@@
 <contactref element="SW2" pad="1B"/>
 <contactref element="R2" pad="2"/>
-<wire x1="5.691" y1="15.756" x2="6.4474" y2="15.756" width="0.6096" layer="1"/>
-<wire x1="3.445" y1="13.51" x2="5.691" y2="15.756" width="0.6096" layer="1"/>
-<wire x1="3.445" y1="5.636" x2="3.445" y2="13.51" width="0.6096" layer="1"/>
+<wire x1="5.691" y1="16.756" x2="6.4474" y2="16.756" width="0.6096" layer="1"/>
+<wire x1="3.445" y1="14.51" x2="5.691" y2="16.756" width="0.6096" layer="1"/>
+<wire x1="3.445" y1="5.636" x2="3.445" y2="14.51" width="0.6096" layer="1"/>
 <contactref element="H1" pad="1"/>
 <wire x1="7.4328" y1="4.7978" x2="7.4328" y2="5.0894" width="0.6096" layer="1"/>
@@
 <contactref element="SW2" pad="0A"/>
 <contactref element="H1" pad="2"/>
-<wire x1="13.4474" y1="10.756" x2="11.9244" y2="10.756" width="0.6096" layer="1"/>
-<wire x1="11.9244" y1="10.756" x2="10.0076" y2="8.8392" width="0.6096" layer="1"/>
+<wire x1="13.4474" y1="11.756" x2="11.9244" y2="11.756" width="0.6096" layer="1"/>
+<wire x1="11.9244" y1="11.756" x2="10.0076" y2="8.8392" width="0.6096" layer="1"/>
 <wire x1="10.0076" y1="8.8392" x2="10.0076" y2="4.8326" width="0.6096" layer="1"/>
 <wire x1="10.0076" y1="4.8326" x2="9.9728" y2="4.7978" width="0.6096" layer="1"/>
