File: Eagle/o8_Relay/Eagle_Relay.brd (EAGLE design)
At the start: 40 x 21.9 mm, 9 parts, among them Q1 S9013, U1 HLS8L-DC3V-S-C

Commit message: miniuno
Changed lines of the file:
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@@
 <setting verticaltext="up"/>
 </settings>
-<grid distance="10" unitdist="mil" unit="mm" style="lines" multiple="1" display="yes" altdistance="0.025" altunitdist="inch" altunit="inch"/>
+<grid distance="10" unitdist="mil" unit="mil" style="lines" multiple="1" display="yes" altdistance="0.025" altunitdist="inch" altunit="inch"/>
 <layers>
 <layer number="1" name="Top" color="4" fill="1" visible="yes" active="yes"/>
@@
 <wire x1="33.2714" y1="1.6176" x2="30.8944" y2="1.6176" width="0.6096" layer="1"/>
 <wire x1="30.8944" y1="1.6176" x2="29.972" y2="2.54" width="0.6096" layer="1"/>
-<via x="29.972" y="2.54" extent="1-16" drill="0.6" shape="square"/>
+<via x="29.972" y="2.54" extent="1-16" drill="0.6"/>
 <wire x1="29.972" y1="2.54" x2="29.972" y2="5.702" width="0.6096" layer="16"/>
 <wire x1="29.972" y1="5.702" x2="33" y2="8.73" width="0.6096" layer="16"/>
 <wire x1="33" y1="8.73" x2="15.842" y2="8.73" width="0.6096" layer="1"/>
 <wire x1="15.842" y1="8.73" x2="14.986" y2="7.874" width="0.6096" layer="1"/>
-<via x="14.986" y="7.874" extent="1-16" drill="0.6" shape="square"/>
+<via x="14.986" y="7.874" extent="1-16" drill="0.5"/>
 <wire x1="14.986" y1="7.874" x2="7.4902" y2="7.874" width="0.6096" layer="16"/>
 <wire x1="7.4902" y1="7.874" x2="7.0254" y2="7.4092" width="0.6096" layer="16"/>
@@
 <wire x1="6.38" y1="1.712" x2="17.46" y2="1.712" width="0.6096" layer="1"/>
 <wire x1="17.46" y1="1.712" x2="18.542" y2="2.54" width="0.6096" layer="1"/>
-<via x="18.542" y="2.54" extent="1-16" drill="0.6" shape="square"/>
+<via x="18.542" y="2.54" extent="1-16" drill="0.5"/>
 <wire x1="18.542" y1="2.54" x2="18.796" y2="2.794" width="0.6096" layer="16"/>
 </signal>

Commit message: 12.15
Parts:
- removed U$7: XMAKERLOGO_2.5MM_TOP, Xmaker_yuhui:XMAKERLOGO_2.5MM_TOP
- added U$8: OPENHARDWARE_5MM_TOP, Xmaker:OPENSOURCE_5MM_TOP
- U$2: value OPENHARDWARE_TOP_2.5MM -> XMAKERLOGO_5MM_TOP; device Xmaker_yuhui:OPENSOURCELOGO_2.5MM -> Xmaker:XMAKERLOGO_5MM_TOP
- moved U$2 10.5 mm to (25.0, 10.0), flipped to the bottom, turned to 0 degrees
Changed lines of the file:
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@@
 <setting verticaltext="up"/>
 </settings>
-<grid distance="10" unitdist="mil" unit="mil" style="lines" multiple="1" display="yes" altdistance="0.025" altunitdist="inch" altunit="inch"/>
+<grid distance="10" unitdist="mil" unit="mm" style="lines" multiple="1" display="yes" altdistance="0.025" altunitdist="inch" altunit="inch"/>
 <layers>
 <layer number="1" name="Top" color="4" fill="1" visible="yes" active="yes"/>
@@
 </element>
 <element name="U$6" library="Xmaker_yuhui" package="DIMENSION_2MM*4MM" value="DIMENSION_4MM2MM" x="0" y="0"/>
-<element name="U$7" library="Xmaker_yuhui" package="XMAKERLOGO_2.5MM_TOP" value="XMAKERLOGO_2.5MM_TOP" x="33.7908" y="3.93" rot="R90"/>
-<element name="U$2" library="Xmaker_yuhui" package="OPENSOURCELOGO_2.5MM" value="OPENHARDWARE_TOP_2.5MM" x="33.528" y="16.1798" rot="R90"/>
 <element name="HEAD_LOCK2" library="Xmaker_yuhuilbr" package="HEAD_LOCK" value="HEAD_LOCK" x="7" y="10" smashed="yes"/>
 <element name="U$3" library="Xmaker_yuhuilbr" package="HEAD_LOCK2" value="HEAD_LOCK2" x="33" y="10" rot="R180"/>
+<element name="U$8" library="Xmaker" package="OPENSOURCE_5MM_TOP" value="OPENHARDWARE_5MM_TOP" x="15" y="10" rot="MR0"/>
+<element name="U$2" library="Xmaker" package="XMAKERLOGO_5MM_TOP" value="XMAKERLOGO_5MM_TOP" x="25" y="10" rot="MR0"/>
 </elements>
 <signals>

Commit message: a
Parts:
- added U$5: NAME_RELAY, Xmaker:NAME_RELAY
- moved U$8 7.65 mm to (22.5, 11.4), turned to 270 degrees
- moved U$2 4.97 mm to (22.5, 5.70), turned to 270 degrees
Changed lines of the file:
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@@
 <?xml version="1.0" encoding="utf-8"?>
 <!DOCTYPE eagle SYSTEM "eagle.dtd">
-<eagle version="6.6.0">
+<eagle version="7.2.0">
 <drawing>
 <settings>
@@
 <pass name="Default">
 <param name="RoutingGrid" value="50mil"/>
+<param name="AutoGrid" value="1"/>
+<param name="Efforts" value="0"/>
+<param name="TopRouterVariant" value="1"/>
 <param name="tpViaShape" value="round"/>
 <param name="PrefDir.1" value="|"/>
@@
 </element>
 <element name="R3" library="Discrete" package="R0603" value="47k" x="34.0334" y="1.6176" smashed="yes" rot="R180">
-<attribute name="NAME" x="32.6364" y="2.246" size="1.016" layer="25" ratio="10" rot="R180"/>
+<attribute name="NAME" x="34.9224" y="3.516" size="1.016" layer="25" ratio="10" rot="R180"/>
 </element>
 <element name="U$6" library="Xmaker_yuhui" package="DIMENSION_2MM*4MM" value="DIMENSION_4MM2MM" x="0" y="0"/>
 <element name="HEAD_LOCK2" library="Xmaker_yuhuilbr" package="HEAD_LOCK" value="HEAD_LOCK" x="7" y="10" smashed="yes"/>
 <element name="U$3" library="Xmaker_yuhuilbr" package="HEAD_LOCK2" value="HEAD_LOCK2" x="33" y="10" rot="R180"/>
-<element name="U$8" library="Xmaker" package="OPENSOURCE_5MM_TOP" value="OPENHARDWARE_5MM_TOP" x="15" y="10" rot="MR0"/>
-<element name="U$2" library="Xmaker" package="XMAKERLOGO_5MM_TOP" value="XMAKERLOGO_5MM_TOP" x="25" y="10" rot="MR0"/>
+<element name="U$8" library="Xmaker" package="OPENSOURCE_5MM_TOP" value="OPENHARDWARE_5MM_TOP" x="22.512" y="11.444" rot="MR270"/>
+<element name="U$2" library="Xmaker" package="XMAKERLOGO_5MM_TOP" value="XMAKERLOGO_5MM_TOP" x="22.512" y="5.696" rot="MR270"/>
+<element name="U$5" library="Xmaker" package="NAME_RELAY" value="NAME_RELAY" x="20.32" y="19.812" rot="MR180"/>
 </elements>
 <signals>
