File: Eagle/o8_Relay/Eagle_Relay.sch (EAGLE design)
At the start: 9 parts, among them J1 Screw Terminal, Q1 S9013, U1 HLS8L-DC3V-S-C

Commit message: lbr
Parts:
- removed HEAD_LOCK1: HEAD_LOCK, Xmaker_yuhui:HEAD_LOCK
- removed J1: Screw Terminal, seeedleo:CON2
- added HEAD_LOCK2: HEAD_LOCK, Xmaker_yuhuilbr:HEAD_LOCK
- added U$3: HEAD_LOCK2, Xmaker_yuhuilbr:HEAD_LOCK2
Connections:
- net COM: now also U$3.2; no longer J1.1
- net D1: now also HEAD_LOCK2.1; no longer HEAD_LOCK1.1
- net GND: now also HEAD_LOCK2.3, U$3.1; no longer HEAD_LOCK1.3, J1.2
- net VCC: now also HEAD_LOCK2.2; no longer HEAD_LOCK1.2
- net VGND: no longer U1.OFF
Changed lines of the file:
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@@
 <part name="Q1" library="Discrete" deviceset="TRANSISTOR-NPN*" device="-SOT23" value="S9013"/>
 <part name="R1" library="Discrete" deviceset="R*" device="-0603" value="4.7k"/>
-<part name="J1" library="seeedleo" deviceset="CON2" device="" value="Screw Terminal"/>
 <part name="U1" library="Seeed" deviceset="RELAY" device="" value="HLS8L-DC3V-S-C"/>
 <part name="U$4" library="moudle" deviceset="SEEEDSTUDIO_SCH_FRAME" device=""/>
 <part name="U$1" library="Power or GND " deviceset="GND_POWER" device=""/>
 <part name="R3" library="Discrete" deviceset="R*" device="-0603" value="47k"/>
-<part name="HEAD_LOCK1" library="Xmaker_yuhui" deviceset="HEAD_LOCK" device=""/>
 <part name="U$6" library="Xmaker_yuhui" deviceset="DIMENSION_4MM*2MM" device=""/>
 <part name="U$7" library="Xmaker_yuhui" deviceset="XMAKERLOGO_2.5MM_TOP" device=""/>
 <part name="U$2" library="Xmaker_yuhui" deviceset="OPENHARDWARE_TOP_2.5MM" device=""/>
+<part name="HEAD_LOCK2" library="Xmaker_yuhuilbr" deviceset="HEAD_LOCK" device=""/>
+<part name="U$3" library="Xmaker_yuhuilbr" deviceset="HEAD_LOCK2" device=""/>
 </parts>
 <sheets>
@@
 <attribute name="VALUE" x="-14.986" y="-22.606" size="1.27" layer="96"/>
 </instance>
-<instance part="J1" gate="CON2" x="49.53" y="-29.21"/>
 <instance part="U1" gate="G$1" x="11.43" y="5.08"/>
 <instance part="U$4" gate="G$1" x="-83.82" y="-104.14"/>
@@
 <attribute name="VALUE" x="-6.096" y="-28.956" size="1.27" layer="96"/>
 </instance>
-<instance part="HEAD_LOCK1" gate="G$1" x="-7.62" y="-40.64"/>
 <instance part="U$6" gate="G$1" x="40.64" y="-45.72"/>
 <instance part="U$7" gate="G$1" x="27.94" y="-45.72"/>
 <instance part="U$2" gate="G$1" x="76.2" y="-45.72"/>
+<instance part="HEAD_LOCK2" gate="G$1" x="-7.62" y="-40.64"/>
+<instance part="U$3" gate="G$1" x="49.276" y="-29.21" rot="R180"/>
 </instances>
 <busses>
@@
 <wire x1="6.35" y1="-43.18" x2="0" y2="-43.18" width="0.1524" layer="91"/>
 <label x="-1.27" y="-43.18" size="1.778" layer="95"/>
-<pinref part="HEAD_LOCK1" gate="G$1" pin="3"/>
+<pinref part="HEAD_LOCK2" gate="G$1" pin="3"/>
 <wire x1="0" y1="-43.18" x2="-1.27" y2="-43.18" width="0.1524" layer="91"/>
 <junction x="0" y="-43.18"/>
@@
 <segment>
 <label x="34.29" y="-30.48" size="1.778" layer="95"/>
-<pinref part="J1" gate="CON2" pin="2"/>
 <wire x1="40.64" y1="-30.48" x2="36.83" y2="-30.48" width="0.1524" layer="91"/>
+<pinref part="U$3" gate="G$1" pin="1"/>
 </segment>
 </net>
@@
 <wire x1="6.35" y1="-40.64" x2="0" y2="-40.64" width="0.1524" layer="91"/>
 <label x="-1.27" y="-40.64" size="1.778" layer="95"/>
-<pinref part="HEAD_LOCK1" gate="G$1" pin="2"/>
+<pinref part="HEAD_LOCK2" gate="G$1" pin="2"/>
 <wire x1="0" y1="-40.64" x2="-1.27" y2="-40.64" width="0.1524" layer="91"/>
 <junction x="0" y="-40.64"/>
@@
 <segment>
 <label x="34.29" y="-27.94" size="1.778" layer="95"/>
-<pinref part="J1" gate="CON2" pin="1"/>
 <wire x1="40.64" y1="-27.94" x2="36.83" y2="-27.94" width="0.1524" layer="91"/>
+<pinref part="U$3" gate="G$1" pin="2"/>
 </segment>
 </net>
 <net name="VGND" class="0">
 <segment>
-<wire x1="3.81" y1="-5.08" x2="3.81" y2="-10.16" width="0.1524" layer="91"/>
-<wire x1="3.81" y1="-10.16" x2="3.81" y2="-15.24" width="0.1524" layer="91"/>
-<wire x1="3.81" y1="-10.16" x2="12.7" y2="-10.16" width="0.1524" layer="91"/>
-<wire x1="12.7" y1="-10.16" x2="13.97" y2="-10.16" width="0.1524" layer="91"/>
-<wire x1="13.97" y1="-10.16" x2="13.97" y2="-15.24" width="0.1524" layer="91"/>
-<junction x="3.81" y="-10.16"/>
-<label x="3.81" y="-12.7" size="1.778" layer="95"/>
+<wire x1="3.81" y1="-5.08" x2="3.81" y2="-15.24" width="0.1524" layer="91"/>
 <pinref part="Q1" gate="Q" pin="C"/>
 <pinref part="U1" gate="G$1" pin="V-"/>
-<pinref part="U1" gate="G$1" pin="OFF"/>
-<wire x1="13.97" y1="-10.16" x2="17.78" y2="-10.16" width="0.1524" layer="91"/>
 </segment>
 </net>
@@
 <label x="0" y="-38.1" size="1.778" layer="95"/>
 <wire x1="6.35" y1="-38.1" x2="0" y2="-38.1" width="0.1524" layer="91"/>
-<pinref part="HEAD_LOCK1" gate="G$1" pin="1"/>
+<pinref part="HEAD_LOCK2" gate="G$1" pin="1"/>
 <wire x1="0" y1="-38.1" x2="-1.27" y2="-38.1" width="0.1524" layer="91"/>
 <junction x="0" y="-38.1"/>

Commit message: 12.15
Parts:
- removed U$7: XMAKERLOGO_2.5MM_TOP, Xmaker_yuhui:XMAKERLOGO_2.5MM_TOP
- added U$8: OPENHARDWARE_5MM_TOP, Xmaker:OPENHARDWARE_5MM_TOP
- U$2: value OPENHARDWARE_TOP_2.5MM -> XMAKERLOGO_5MM_TOP; device Xmaker_yuhui:OPENHARDWARE_TOP_2.5MM -> Xmaker:XMAKERLOGO_5MM_TOP
Changed lines of the file:
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@@
 <setting verticaltext="up"/>
 </settings>
-<grid distance="10" unitdist="mil" unit="mil" style="lines" multiple="1" display="no" altdistance="0.01" altunitdist="inch" altunit="inch"/>
+<grid distance="0.1" unitdist="inch" unit="inch" style="lines" multiple="1" display="no" altdistance="0.01" altunitdist="inch" altunit="inch"/>
 <layers>
 <layer number="1" name="Top" color="4" fill="1" visible="no" active="no"/>
@@
 <part name="R3" library="Discrete" deviceset="R*" device="-0603" value="47k"/>
 <part name="U$6" library="Xmaker_yuhui" deviceset="DIMENSION_4MM*2MM" device=""/>
-<part name="U$7" library="Xmaker_yuhui" deviceset="XMAKERLOGO_2.5MM_TOP" device=""/>
-<part name="U$2" library="Xmaker_yuhui" deviceset="OPENHARDWARE_TOP_2.5MM" device=""/>
 <part name="HEAD_LOCK2" library="Xmaker_yuhuilbr" deviceset="HEAD_LOCK" device=""/>
 <part name="U$3" library="Xmaker_yuhuilbr" deviceset="HEAD_LOCK2" device=""/>
+<part name="U$8" library="Xmaker" deviceset="OPENHARDWARE_5MM_TOP" device=""/>
+<part name="U$2" library="Xmaker" deviceset="XMAKERLOGO_5MM_TOP" device=""/>
 </parts>
 <sheets>
@@
 </instance>
 <instance part="U$6" gate="G$1" x="40.64" y="-45.72"/>
-<instance part="U$7" gate="G$1" x="27.94" y="-45.72"/>
-<instance part="U$2" gate="G$1" x="76.2" y="-45.72"/>
 <instance part="HEAD_LOCK2" gate="G$1" x="-7.62" y="-40.64"/>
 <instance part="U$3" gate="G$1" x="49.276" y="-29.21" rot="R180"/>
+<instance part="U$8" gate="G$1" x="63.5" y="-55.88"/>
+<instance part="U$2" gate="G$1" x="30.48" y="-53.34"/>
 </instances>
 <busses>

Commit message: a
Parts:
- added U$5: NAME_RELAY, Xmaker:NAME_RELAY
Changed lines of the file:
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@@
 <?xml version="1.0" encoding="utf-8"?>
 <!DOCTYPE eagle SYSTEM "eagle.dtd">
-<eagle version="6.6.0">
+<eagle version="7.2.0">
 <drawing>
 <settings>
@@
 <part name="U$8" library="Xmaker" deviceset="OPENHARDWARE_5MM_TOP" device=""/>
 <part name="U$2" library="Xmaker" deviceset="XMAKERLOGO_5MM_TOP" device=""/>
+<part name="U$5" library="Xmaker" deviceset="NAME_RELAY" device=""/>
 </parts>
 <sheets>
@@
 <instance part="U$8" gate="G$1" x="63.5" y="-55.88"/>
 <instance part="U$2" gate="G$1" x="30.48" y="-53.34"/>
+<instance part="U$5" gate="G$1" x="5.08" y="-53.34"/>
 </instances>
 <busses>
