File: Eagle/f7_General/f7_General.brd (EAGLE design)
At the start: 160 x 100.3 mm, 14 parts, among them IC1 TINY13-20SSU

Commit message: dd
Parts:
- moved LED1 79.0 mm to (42.2, 24.1), turned to 180 degrees
- moved R2 77.7 mm to (42.2, 25.4)
- moved R1 69.7 mm to (21.3, 3.81), turned to 90 degrees
- moved C1 65.8 mm to (31.5, 13.7)
- moved U$5 3.06 mm to (28.4, 16.8)
- moved S1 1.61 mm to (29.0, 3.05)
Changed lines of the file:
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@@
 </autorouter>
 <elements>
-<element name="IC1" library="atmel" package="8S1" value="TINY13-20SSU" x="27.94" y="10.16" rot="R270">
+<element name="IC1" library="atmel" package="8S1" value="TINY13-20SSU" x="27.94" y="10.16" smashed="yes" rot="R270">
 <attribute name="OC_NEWARK" value="58M3771" x="64.77" y="26.67" size="1.778" layer="27" rot="R270" display="off"/>
 <attribute name="MPN" value="ATTINY13-20SSU" x="64.77" y="26.67" size="1.778" layer="27" rot="R270" display="off"/>
 <attribute name="MF" value="" x="64.77" y="26.67" size="1.778" layer="27" rot="R270" display="off"/>
 <attribute name="OC_FARNELL" value="1455133" x="64.77" y="26.67" size="1.778" layer="27" rot="R270" display="off"/>
+<attribute name="NAME" x="25.781" y="13.0175" size="1.27" layer="25" ratio="10"/>
 </element>
-<element name="C1" library="SparkFun-Passives" package="0603-CAP" value="0.1uF" x="33.02" y="-52.07"/>
-<element name="R2" library="SparkFun-Resistors" package="0603-RES" value="" x="36.83" y="-52.07">
-<attribute name="PROD_ID" value="RES-08787" x="2.54" y="-15.24" size="1.778" layer="27" display="off"/>
+<element name="C1" library="SparkFun-Passives" package="0603-CAP" value="0.1uF" x="31.496" y="13.716" smashed="yes">
+<attribute name="NAME" x="30.607" y="14.478" size="0.8128" layer="25" font="vector"/>
+<attribute name="VALUE" x="30.48" y="12.573" size="0.8128" layer="27" font="vector"/>
 </element>
-<element name="LED1" library="eagle-ltspice" package="LED_SML0603" value="" x="26.67" y="-53.34">
-<attribute name="SPICEMODEL" value="NONE" x="2.54" y="-19.05" size="1.778" layer="27" display="off"/>
-<attribute name="SPICETYPE" value="diode" x="2.54" y="-19.05" size="1.778" layer="27" display="off"/>
-<attribute name="SPICEPREFIX" value="D" x="2.54" y="-19.05" size="1.778" layer="27" display="off"/>
+<element name="R2" library="SparkFun-Resistors" package="0603-RES" value="" x="42.164" y="25.4" smashed="yes">
+<attribute name="PROD_ID" value="RES-08787" x="7.874" y="62.23" size="1.778" layer="27" display="off"/>
+<attribute name="NAME" x="41.529" y="26.162" size="0.8128" layer="25" font="vector"/>
+<attribute name="VALUE" x="41.148" y="24.257" size="0.4064" layer="27" font="vector"/>
+</element>
+<element name="LED1" library="eagle-ltspice" package="LED_SML0603" value="" x="42.164" y="24.13" smashed="yes" rot="R180">
+<attribute name="SPICEMODEL" value="NONE" x="66.294" y="-10.16" size="1.778" layer="27" rot="R180" display="off"/>
+<attribute name="SPICETYPE" value="diode" x="66.294" y="-10.16" size="1.778" layer="27" rot="R180" display="off"/>
+<attribute name="SPICEPREFIX" value="D" x="66.294" y="-10.16" size="1.778" layer="27" rot="R180" display="off"/>
+<attribute name="NAME" x="43.672" y="23.638" size="0.8128" layer="25" rot="R180"/>
+<attribute name="VALUE" x="43.164" y="26.13" size="1.27" layer="27" rot="R180"/>
 </element>
 <element name="U$3" library="Xmaker_yuhui" package="DIMENSION1" value="DIMENSION1" x="0" y="0"/>
 <element name="U$2" library="Xmaker_yuhui" package="XMAKERLOGO_5MM_TOP" value="XMAKERLOGO_5MM_TOP" x="16.51" y="-57.15"/>
 <element name="U$4" library="Xmaker_yuhui" package="OPENSOURCE_5MM_TOP" value="OPENHARDWARE_5MM_TOP" x="21.59" y="-53.34"/>
-<element name="U$5" library="Xmaker" package="POT_CIRCLE" value="POL_CIRCLE" x="25.4" y="16.51"/>
+<element name="U$5" library="Xmaker" package="POT_CIRCLE" value="POL_CIRCLE" x="28.448" y="16.764"/>
 <element name="HEAD_LOCK1" library="Xmaker" package="HEAD_LOCK_3PIN_3" value="HEAD_LOCK_3PIN_3" x="10.16" y="22.352" rot="R270"/>
 <element name="HEAD_LOCK2" library="Xmaker" package="HEAD_LOCK_3PIN_3" value="HEAD_LOCK_3PIN_3" x="42.418" y="14.986" rot="R180"/>
-<element name="S1" library="SparkFun-Electromechanical" package="SWITCH-SPDT_KIT" value="" x="30.48" y="2.54" rot="R90">
-<attribute name="PROD_ID" value="SWCH-08261" x="10.16" y="-10.16" size="1.778" layer="27" rot="R90" display="off"/>
+<element name="S1" library="SparkFun-Electromechanical" package="SWITCH-SPDT_KIT" value="" x="28.956" y="3.048" smashed="yes" rot="R90">
+<attribute name="PROD_ID" value="SWCH-08261" x="8.636" y="-9.652" size="1.778" layer="27" rot="R90" display="off"/>
+<attribute name="NAME" x="35.306" y="4.572" size="1.27" layer="25" ratio="10" rot="SR270"/>
+<attribute name="VALUE" x="38.481" y="-0.762" size="1.778" layer="27" ratio="10" rot="R90"/>
 </element>
-<element name="R1" library="SparkFun-Passives" package="0603-RES" value="" x="8.89" y="-64.77"/>
+<element name="R1" library="SparkFun-Passives" package="0603-RES" value="" x="21.336" y="3.81" smashed="yes" rot="R90">
+<attribute name="NAME" x="20.574" y="3.175" size="0.8128" layer="25" font="vector" rot="R90"/>
+<attribute name="VALUE" x="22.479" y="2.794" size="0.4064" layer="27" font="vector" rot="R90"/>
+</element>
 <element name="HEAD_LOCK3" library="Xmaker" package="HEAD_LOCK_3PIN_3" value="HEAD_LOCK_3PIN_3" x="7.62" y="14.986" smashed="yes">
 <attribute name="NAME" x="10.118" y="10.7478" size="0.8128" layer="21" rot="R90"/>
@@
 <contactref element="HEAD_LOCK4" pad="2"/>
 <contactref element="R1" pad="2"/>
-<wire x1="27.42" y1="-53.34" x2="9.74" y2="-64.77" width="0" layer="19" extent="1-1"/>
-<wire x1="32.17" y1="-52.07" x2="27.42" y2="-53.34" width="0" layer="19" extent="1-1"/>
-<wire x1="30.594" y1="12.065" x2="32.17" y2="-52.07" width="0" layer="19" extent="1-1"/>
+<wire x1="41.414" y1="24.13" x2="21.336" y2="4.66" width="0" layer="19" extent="1-1"/>
+<wire x1="30.646" y1="13.716" x2="41.414" y2="24.13" width="0" layer="19" extent="1-1"/>
+<wire x1="30.594" y1="12.065" x2="30.646" y2="13.716" width="0" layer="19" extent="1-1"/>
 <wire x1="25.286" y1="12.065" x2="30.594" y2="12.065" width="0" layer="19" extent="1-1"/>
-<wire x1="21.4" y1="16.51" x2="25.286" y2="12.065" width="0" layer="19" extent="1-1"/>
+<wire x1="24.448" y1="16.764" x2="25.286" y2="12.065" width="0" layer="19" extent="1-1"/>
 <wire x1="42.3926" y1="15.0368" x2="30.594" y2="12.065" width="0" layer="19" extent="1-1"/>
-<wire x1="10.1092" y1="22.3266" x2="21.4" y2="16.51" width="0" layer="19" extent="1-1"/>
+<wire x1="10.1092" y1="22.3266" x2="24.448" y2="16.764" width="0" layer="19" extent="1-1"/>
 <wire x1="7.6454" y1="14.9352" x2="10.1092" y2="22.3266" width="0" layer="19" extent="1-1"/>
 <wire x1="10.2108" y1="7.6454" x2="7.6454" y2="14.9352" width="0" layer="19" extent="1-1"/>
@@
 <contactref element="HEAD_LOCK4" pad="3"/>
 <contactref element="S1" pad="3"/>
-<wire x1="29.4" y1="16.51" x2="42.3926" y2="17.5768" width="0" layer="19" extent="1-1"/>
-<wire x1="25.286" y1="8.265" x2="29.4" y2="16.51" width="0" layer="19" extent="1-1"/>
-<wire x1="33.1978" y1="2.54" x2="25.286" y2="8.265" width="0" layer="19" extent="1-1"/>
+<wire x1="32.448" y1="16.764" x2="42.3926" y2="17.5768" width="0" layer="19" extent="1-1"/>
+<wire x1="25.286" y1="8.265" x2="32.448" y2="16.764" width="0" layer="19" extent="1-1"/>
+<wire x1="31.6738" y1="3.048" x2="25.286" y2="8.265" width="0" layer="19" extent="1-1"/>
 <wire x1="12.7508" y1="7.6454" x2="25.286" y2="8.265" width="0" layer="19" extent="1-1"/>
 <wire x1="7.6454" y1="12.3952" x2="12.7508" y2="7.6454" width="0" layer="19" extent="1-1"/>
 <wire x1="7.5692" y1="22.3266" x2="7.6454" y2="12.3952" width="0" layer="19" extent="1-1"/>
-<wire x1="33.87" y1="-52.07" x2="33.1978" y2="2.54" width="0" layer="19" extent="1-1"/>
-<wire x1="35.98" y1="-52.07" x2="33.87" y2="-52.07" width="0" layer="19" extent="1-1"/>
+<wire x1="32.346" y1="13.716" x2="31.6738" y2="3.048" width="0" layer="19" extent="1-1"/>
+<wire x1="41.314" y1="25.4" x2="32.346" y2="13.716" width="0" layer="19" extent="1-1"/>
 </signal>
 <signal name="CONTROL">
 <contactref element="U$5" pad="P$2"/>
 <contactref element="IC1" pad="6"/>
-<wire x1="30.594" y1="9.525" x2="25.4" y2="16.51" width="0" layer="19" extent="1-1"/>
+<wire x1="30.594" y1="9.525" x2="28.448" y2="16.764" width="0" layer="19" extent="1-1"/>
 </signal>
 <signal name="N$1">
 <contactref element="R2" pad="2"/>
 <contactref element="LED1" pad="C"/>
-<wire x1="37.68" y1="-52.07" x2="25.92" y2="-53.34" width="0" layer="19" extent="1-1"/>
+<wire x1="43.014" y1="25.4" x2="42.914" y2="24.13" width="0" layer="19" extent="1-1"/>
 </signal>
 <signal name="N$2">
 <contactref element="R1" pad="1"/>
 <contactref element="S1" pad="1"/>
-<wire x1="8.04" y1="-64.77" x2="27.7622" y2="2.54" width="0" layer="19" extent="1-1"/>
+<wire x1="21.336" y1="2.96" x2="26.2382" y2="3.048" width="0" layer="19" extent="1-1"/>
 </signal>
 <signal name="SELECT">
 <contactref element="S1" pad="2"/>
 <contactref element="IC1" pad="7"/>
-<wire x1="30.594" y1="10.795" x2="30.48" y2="2.54" width="0" layer="19" extent="1-1"/>
+<wire x1="30.594" y1="10.795" x2="28.956" y2="3.048" width="0" layer="19" extent="1-1"/>
 </signal>
 <signal name="IN1">
