File: Eagle/f1_Not/f1_Not.brd (EAGLE design)
At the start: 160 x 100 mm, 8 parts, among them IC2 TINY13-20SSU

Commit message: d
Parts:
- added U$3: (no value), Xmaker:NAME_ANALOG
Changed lines of the file:
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@@
 <?xml version="1.0" encoding="utf-8"?>
 <!DOCTYPE eagle SYSTEM "eagle.dtd">
-<eagle version="6.6.0">
+<eagle version="7.2.0">
 <drawing>
 <settings>
@@
 <pass name="Default">
 <param name="RoutingGrid" value="50mil"/>
+<param name="AutoGrid" value="1"/>
+<param name="Efforts" value="0"/>
+<param name="TopRouterVariant" value="1"/>
 <param name="tpViaShape" value="round"/>
 <param name="PrefDir.1" value="|"/>
@@
 <element name="U$1" library="Xmaker_yuhui" package="DIMENSION1" value="DIMENSION1" x="35.56" y="26.67"/>
 <element name="U$2" library="SparkFun-Aesthetics" package="OSHW-LOGO-M" value="" x="73.406" y="52.07"/>
+<element name="U$3" library="Xmaker" package="NAME_ANALOG" value="" x="60.452" y="27.7876"/>
 </elements>
 <signals>
