File: Eagle/i5_Light/Version2/i5_Light_Ver2/Light.brd (EAGLE design)
At the start: 160 x 100 mm, 6 parts, among them IC1 LM358D

Commit message: light
Parts:
- removed I15SW1: (no value), SparkFun:AYZ0202
- added R2: (no value), Discrete:3P-SQUA-7X6.8
- added U$1: DIMENSION_2MM2MM, Xmaker:DIMENSION_2MM*2MM
- added U$2: NAME_LIGHT, Xmaker:NAME_LIGHT
- added U$3: OPENHARDWARE_2.5MM_TOP, Xmaker:OPENSOURCELOGO_2.5MM
- added U$4: XMAKERLOGO_2.5MM_TOP, Xmaker:XMAKERLOGO_2.5MM_TOP
- added U$5: MSS-22C02, Xmaker:MSS-22C02
- H1: value HEAD_LOCK -> HEAD_LOCK_3PIN_2; device HEAD_LOCK:HEAD_LOCK -> Xmaker:HEAD_LOCK_3PIN_2
- moved I15C1 51.6 mm to (30.8, 14.2), flipped to the bottom
- moved H1 47.7 mm to (24.1, 11.3), turned to 90 degrees
- moved LIGHT 45.1 mm to (26.6, 24.3), turned to 270 degrees
- moved R1 44.0 mm to (20.2, 23.9)
- moved IC1 35.6 mm to (27.4, 18.4), flipped to the bottom, turned to 270 degrees
Connections:
- removed net V+: IC1.8
- removed net V-: IC1.4
- new net N$5: IC1.6, U$5.3, U$5.6
- net GND: now also IC1.4, R1.1, R2.2
- net N$1: now also U$5.2; no longer I15SW1.2
- net N$3: now also U$5.1, U$5.4; no longer I15SW1.1, I15SW1.6, IC1.5
- net N$4: now also R2.3, U$5.5; no longer I15SW1.3, I15SW1.4, IC1.6
- net VCC: now also IC1.8, R2.1
Routing:
- net VCC: track 0.00 -> 39.3 mm
- net OUT: track 0.00 -> 10.3 mm
- net GND: track 0.00 -> 9.17 mm
- net N$2: track 0.00 -> 4.39 mm
- net N$1: track 0.00 -> 1.27 mm

Commit message: d
Parts:
- moved U$4 88.5 mm to (21.8, 21.4), flipped to the bottom, turned to 270 degrees
- moved U$2 73.8 mm to (13.8, 12.5), turned to 270 degrees
- moved U$3 22.0 mm to (22.2, 24.6), flipped to the bottom, turned to 270 degrees
- moved U$5 7.50 mm to (30.2, 16.2), turned to 180 degrees
Connections:
- net N$3: now also IC1.5
Routing:
- net N$3: track 0.00 -> 25.3 mm, vias 0 -> 1
- net GND: track 9.17 -> 32.9 mm
- net N$2: track 4.39 -> 21.6 mm
- net N$5: track 0.00 -> 14.7 mm, vias 0 -> 1
- net N$4: track 0.00 -> 7.90 mm
- net N$1: track 1.27 -> 6.04 mm, vias 0 -> 1
- net VCC: track 39.3 -> 38.4 mm
- added copper zone on layer 1, net GND
- added copper zone on layer 16, net GND
Changed lines of the file:
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@@
 </element>
 <element name="U$1" library="Xmaker" package="DIMENSION_2MM*2MM" value="DIMENSION_2MM2MM" x="13.97" y="6.35"/>
-<element name="U$2" library="Xmaker" package="NAME_LIGHT" value="NAME_LIGHT" x="-13.97" y="-55.88"/>
-<element name="U$3" library="Xmaker" package="OPENSOURCELOGO_2.5MM" value="OPENHARDWARE_2.5MM_TOP" x="40.0304" y="11.7348"/>
-<element name="U$4" library="Xmaker" package="XMAKERLOGO_2.5MM_TOP" value="XMAKERLOGO_2.5MM_TOP" x="-19.05" y="-57.15"/>
-<element name="U$5" library="Xmaker" package="MSS-22C02" value="MSS-22C02" x="24.5872" y="21.1328" smashed="yes"/>
+<element name="U$2" library="Xmaker" package="NAME_LIGHT" value="NAME_LIGHT" x="13.843" y="12.4714" rot="R270"/>
+<element name="U$3" library="Xmaker" package="OPENSOURCELOGO_2.5MM" value="OPENHARDWARE_2.5MM_TOP" x="22.1742" y="24.5618" rot="MR270"/>
+<element name="U$4" library="Xmaker" package="XMAKERLOGO_2.5MM_TOP" value="XMAKERLOGO_2.5MM_TOP" x="21.8186" y="21.3614" rot="MR270"/>
+<element name="U$5" library="Xmaker" package="MSS-22C02" value="MSS-22C02" x="30.2006" y="16.1544" rot="R180"/>
 </elements>
 <signals>
@@
 <wire x1="25.3746" y1="9.6266" x2="24.13" y2="10.8712" width="0.6096" layer="16"/>
 <wire x1="24.13" y1="10.8712" x2="24.13" y2="11.2522" width="0.6096" layer="16"/>
-<wire x1="24.7558" y1="20.3454" x2="24.7812" y2="20.3708" width="0.4064" layer="16"/>
-<wire x1="24.7812" y1="20.3708" x2="26.6192" y2="20.3708" width="0.4064" layer="16"/>
-<wire x1="26.6192" y1="20.3708" x2="27.8638" y2="21.6154" width="0.4064" layer="16"/>
-<wire x1="27.8638" y1="21.6154" x2="27.8638" y2="24.2824" width="0.4064" layer="16"/>
 <wire x1="19.3" y1="16.51" x2="19.3294" y2="16.5394" width="0.6096" layer="16"/>
 <wire x1="19.3294" y1="16.5394" x2="19.3294" y2="18.3134" width="0.6096" layer="16"/>
 <wire x1="19.3294" y1="18.3134" x2="21.3614" y2="20.3454" width="0.6096" layer="16"/>
 <wire x1="21.3614" y1="20.3454" x2="24.7558" y2="20.3454" width="0.6096" layer="16"/>
+<wire x1="24.7558" y1="20.3454" x2="25.4762" y2="20.3454" width="0.6096" layer="16"/>
+<wire x1="25.4762" y1="20.3454" x2="26.4414" y2="21.4122" width="0.6096" layer="16"/>
+<wire x1="26.4414" y1="21.4122" x2="27.8638" y2="24.2824" width="0.6096" layer="16"/>
 </signal>
 <signal name="N$1">
 <contactref element="IC1" pad="1"/>
 <contactref element="IC1" pad="2"/>
+<wire x1="29.9558" y1="19.0754" x2="29.9558" y2="20.3454" width="0.6096" layer="16"/>
 <contactref element="U$5" pad="2"/>
-<wire x1="29.9558" y1="19.0754" x2="24.5872" y2="18.5928" width="0" layer="19" extent="1-16"/>
-<wire x1="29.9558" y1="19.0754" x2="29.9558" y2="20.3454" width="0.6096" layer="16"/>
+<wire x1="30.2006" y1="18.6944" x2="30.226" y2="18.669" width="0.4064" layer="1"/>
+<wire x1="30.226" y1="18.669" x2="31.4706" y2="18.669" width="0.4064" layer="1"/>
+<wire x1="31.4706" y1="18.669" x2="31.7754" y2="18.9738" width="0.4064" layer="1"/>
+<wire x1="31.7754" y1="18.9738" x2="31.7754" y2="19.5326" width="0.4064" layer="1"/>
+<via x="31.7754" y="19.5326" extent="1-16" drill="0.6096"/>
+<wire x1="31.7754" y1="19.5326" x2="31.7754" y2="20.1168" width="0.4064" layer="16"/>
+<wire x1="31.7754" y1="20.1168" x2="31.5468" y2="20.3454" width="0.4064" layer="16"/>
+<wire x1="31.5468" y1="20.3454" x2="30.6324" y2="20.3454" width="0.4064" layer="16"/>
+<wire x1="30.6324" y1="20.3454" x2="29.9558" y2="20.3454" width="0.254" layer="16"/>
 </signal>
 <signal name="N$2">
@@
 <contactref element="LIGHT" pad="2"/>
 <contactref element="R1" pad="2"/>
-<wire x1="29.9558" y1="17.8054" x2="25.3238" y2="24.2824" width="0" layer="19" extent="1-1"/>
 <wire x1="21.082" y1="23.9268" x2="23.0378" y2="23.9268" width="0.6096" layer="1"/>
 <wire x1="23.0378" y1="23.9268" x2="23.3934" y2="24.2824" width="0.6096" layer="1"/>
 <wire x1="23.3934" y1="24.2824" x2="25.3238" y2="24.2824" width="0.6096" layer="1"/>
+<wire x1="25.3238" y1="24.2824" x2="26.67" y2="25.6286" width="0.6096" layer="16"/>
+<wire x1="26.67" y1="25.6286" x2="29.0576" y2="25.6286" width="0.6096" layer="16"/>
+<wire x1="29.0576" y1="25.6286" x2="30.0482" y2="24.638" width="0.6096" layer="16"/>
+<wire x1="30.0482" y1="24.638" x2="30.0482" y2="23.2918" width="0.6096" layer="16"/>
+<wire x1="30.0482" y1="23.2918" x2="30.8356" y2="22.5044" width="0.6096" layer="16"/>
+<wire x1="30.8356" y1="22.5044" x2="32.2072" y2="22.5044" width="0.6096" layer="16"/>
+<wire x1="32.2072" y1="22.5044" x2="32.9946" y2="21.717" width="0.6096" layer="16"/>
+<wire x1="32.9946" y1="21.717" x2="33.1216" y2="18.8722" width="0.6096" layer="16"/>
+<wire x1="33.1216" y1="18.8722" x2="32.0294" y2="17.78" width="0.6096" layer="16"/>
+<wire x1="32.0294" y1="17.78" x2="29.8704" y2="17.8054" width="0.6096" layer="16"/>
+<wire x1="29.8704" y1="17.8054" x2="29.9558" y2="17.8054" width="0" layer="19" extent="16-16"/>
 </signal>
 <signal name="GND">
@@
 <contactref element="R2" pad="2"/>
 <contactref element="R1" pad="1"/>
-<wire x1="19.3" y1="21.59" x2="29.9348" y2="14.1986" width="0" layer="19" extent="16-16"/>
 <wire x1="19.3" y1="21.59" x2="19.304" y2="21.594" width="0.6096" layer="1"/>
 <wire x1="19.304" y1="21.594" x2="19.304" y2="23.9268" width="0.6096" layer="1"/>
@@
 <wire x1="29.9348" y1="14.1986" x2="26.9884" y2="11.2522" width="0.6096" layer="16"/>
 <wire x1="26.9884" y1="11.2522" x2="26.67" y2="11.2522" width="0.6096" layer="16"/>
+<wire x1="19.3" y1="21.59" x2="16.51" y2="21.59" width="0.6096" layer="1"/>
+<wire x1="16.51" y1="21.59" x2="15.3924" y2="20.4724" width="0.6096" layer="1"/>
+<wire x1="15.3924" y1="20.4724" x2="15.3924" y2="13.462" width="0.6096" layer="1"/>
+<wire x1="15.3924" y1="13.462" x2="16.2306" y2="12.6238" width="0.6096" layer="1"/>
+<wire x1="16.2306" y1="12.6238" x2="25.6032" y2="12.6238" width="0.6096" layer="1"/>
+<wire x1="25.6032" y1="12.6238" x2="26.67" y2="11.557" width="0.6096" layer="1"/>
+<wire x1="26.67" y1="11.557" x2="26.67" y2="11.2522" width="0.6096" layer="1"/>
+<polygon width="0.3048" layer="1" isolate="0.6096">
+<vertex x="12.8778" y="27.4828"/>
+<vertex x="35.814" y="27.4828"/>
+<vertex x="35.814" y="3.2004"/>
+<vertex x="12.827" y="3.2004"/>
+<vertex x="12.827" y="27.5082"/>
+</polygon>
+<polygon width="0.3048" layer="16" isolate="0.6096">
+<vertex x="12.9286" y="27.5336"/>
+<vertex x="35.8394" y="27.5336"/>
+<vertex x="35.8394" y="3.175"/>
+<vertex x="12.9286" y="3.175"/>
+</polygon>
 </signal>
 <signal name="OUT">
@@
 <wire x1="21.59" y1="17.907" x2="21.59" y2="11.2522" width="0.6096" layer="16"/>
 </signal>
-<signal name="N$3">
-<contactref element="U$5" pad="1"/>
-<contactref element="U$5" pad="4"/>
-<wire x1="30.2372" y1="16.0528" x2="24.5872" y2="21.1328" width="0" layer="19" extent="1-1"/>
-</signal>
 <signal name="N$5">
+<contactref element="IC1" pad="6"/>
 <contactref element="U$5" pad="3"/>
-<contactref element="IC1" pad="6"/>
 <contactref element="U$5" pad="6"/>
-<wire x1="24.5872" y1="16.0528" x2="30.2372" y2="21.1328" width="0" layer="19" extent="1-1"/>
-<wire x1="24.7558" y1="17.8054" x2="24.5872" y2="16.0528" width="0" layer="19" extent="1-16"/>
+<wire x1="24.5506" y1="16.1544" x2="28.1686" y2="16.1544" width="0.4064" layer="1"/>
+<wire x1="28.1686" y1="16.1544" x2="28.7782" y2="16.764" width="0.4064" layer="1"/>
+<wire x1="28.7782" y1="16.764" x2="28.7782" y2="20.828" width="0.4064" layer="1"/>
+<wire x1="28.7782" y1="20.828" x2="29.0576" y2="21.1074" width="0.4064" layer="1"/>
+<wire x1="29.0576" y1="21.1074" x2="30.0736" y2="21.1074" width="0.4064" layer="1"/>
+<wire x1="30.0736" y1="21.1074" x2="30.2006" y2="21.2344" width="0.4064" layer="1"/>
+<wire x1="24.7558" y1="17.8054" x2="23.4188" y2="17.8054" width="0.254" layer="16"/>
+<wire x1="23.4188" y1="17.8054" x2="22.86" y2="17.2466" width="0.254" layer="16"/>
+<via x="22.86" y="17.2466" extent="1-16" drill="0.6096"/>
+<wire x1="22.86" y1="17.2466" x2="22.86" y2="16.6624" width="0.254" layer="1"/>
+<wire x1="22.86" y1="16.6624" x2="23.368" y2="16.1544" width="0.254" layer="1"/>
+<wire x1="23.368" y1="16.1544" x2="24.5506" y2="16.1544" width="0.254" layer="1"/>
 </signal>
 <signal name="N$4">
 <contactref element="R2" pad="3"/>
 <contactref element="U$5" pad="5"/>
-<wire x1="16.8" y1="19.05" x2="30.2372" y2="18.5928" width="0" layer="19" extent="1-1"/>
+<wire x1="24.5506" y1="18.6944" x2="17.1556" y2="18.6944" width="0.6096" layer="1"/>
+<wire x1="17.1556" y1="18.6944" x2="16.8" y2="19.05" width="0.6096" layer="1"/>
+</signal>
+<signal name="N$3">
+<contactref element="U$5" pad="1"/>
+<contactref element="U$5" pad="4"/>
+<wire x1="24.5506" y1="21.2344" x2="24.638" y2="21.3218" width="0.6096" layer="1"/>
+<wire x1="24.638" y1="21.3218" x2="24.638" y2="22.1742" width="0.6096" layer="1"/>
+<wire x1="24.638" y1="22.1742" x2="25.0444" y2="22.5806" width="0.6096" layer="1"/>
+<wire x1="25.0444" y1="22.5806" x2="31.496" y2="22.5806" width="0.6096" layer="1"/>
+<wire x1="31.496" y1="22.5806" x2="32.8168" y2="21.2598" width="0.6096" layer="1"/>
+<wire x1="32.8168" y1="21.2598" x2="32.8168" y2="16.9418" width="0.6096" layer="1"/>
+<wire x1="32.8168" y1="16.9418" x2="32.0294" y2="16.1544" width="0.6096" layer="1"/>
+<wire x1="32.0294" y1="16.1544" x2="30.2006" y2="16.1544" width="0.6096" layer="1"/>
+<contactref element="IC1" pad="5"/>
+<wire x1="24.7558" y1="16.5354" x2="26.0604" y2="16.5354" width="0.6096" layer="16"/>
+<wire x1="26.0604" y1="16.5354" x2="26.8986" y2="15.6972" width="0.6096" layer="16"/>
+<wire x1="26.8986" y1="15.6972" x2="26.8986" y2="14.5542" width="0.6096" layer="16"/>
+<via x="26.8986" y="14.5542" extent="1-16" drill="0.6096"/>
+<wire x1="26.8986" y1="14.5542" x2="29.6164" y2="14.5542" width="0.6096" layer="1"/>
+<wire x1="29.6164" y1="14.5542" x2="30.2006" y2="15.1384" width="0.6096" layer="1"/>
+<wire x1="30.2006" y1="15.1384" x2="30.2006" y2="16.1544" width="0.6096" layer="1"/>
 </signal>
 </signals>
