File: Eagle/i5_Light/Version2/i5_Light_Ver2/Light.sch (EAGLE design)
At the start: 6 parts, among them IC1 LM358D

Commit message: light
Parts:
- removed I15SW1: SWITCH-DPDTSMD, SparkFun:SWITCH-DPDTSMD
- added R2: (no value), Discrete:R-POTENTIOMETER3362
- added U$1: DIMENSION_2MM2MM, Xmaker:DIMENSION_2MM2MM
- added U$2: NAME_LIGHT, Xmaker:NAME_LIGHT
- added U$3: OPENHARDWARE_2.5MM_TOP, Xmaker:OPENHARDWARE_2.5MM_TOP
- added U$4: XMAKERLOGO_2.5MM_TOP, Xmaker:XMAKERLOGO_2.5MM_TOP
- added U$5: MSS-22C02, Xmaker:MSS-22C02
- H1: value HEAD_LOCK -> HEAD_LOCK_3PIN_2; device HEAD_LOCK:HEAD_LOCK -> Xmaker:HEAD_LOCK_3PIN_2
Connections:
- new net N$5: IC1B.-IN, U$5.3, U$5.6
- net GND: now also IC1P.V-, R1.1, R2.2
- net N$1: now also U$5.2; no longer I15SW1.2
- net N$3: now also U$5.1, U$5.4; no longer I15SW1.1, I15SW1.6, IC1B.+IN
- net N$4: now also R2.3, U$5.5; no longer I15SW1.3, I15SW1.4, IC1B.-IN
- net VCC: now also IC1P.V+, R2.1
Other:
- moved on the sheet: H1, I15C1

Commit message: d
Connections:
- net N$3: now also IC1B.+IN
Changed lines of the file:
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@@
 <instance part="U$3" gate="G$1" x="17.018" y="-34.29"/>
 <instance part="U$4" gate="G$1" x="33.274" y="-34.29"/>
-<instance part="U$5" gate="G$1" x="4.572" y="23.114"/>
+<instance part="U$5" gate="G$1" x="7.112" y="23.114"/>
 </instances>
 <busses>
@@
 <wire x1="-9.398" y1="7.874" x2="-9.398" y2="19.304" width="0.1524" layer="91"/>
 <junction x="-9.398" y="19.304"/>
+<wire x1="-9.398" y1="20.574" x2="-9.398" y2="19.304" width="0.1524" layer="91"/>
+<wire x1="-0.508" y1="20.574" x2="-9.398" y2="20.574" width="0.1524" layer="91"/>
 <pinref part="U$5" gate="G$1" pin="2"/>
-<wire x1="-9.398" y1="20.574" x2="-9.398" y2="19.304" width="0.1524" layer="91"/>
-<wire x1="-3.048" y1="20.574" x2="-9.398" y2="20.574" width="0.1524" layer="91"/>
 </segment>
 </net>
@@
 <net name="N$3" class="0">
 <segment>
-<pinref part="U$5" gate="G$1" pin="1"/>
-<wire x1="-3.048" y1="23.114" x2="-4.826" y2="23.114" width="0.1524" layer="91"/>
+<wire x1="-0.508" y1="23.114" x2="-4.826" y2="23.114" width="0.1524" layer="91"/>
 <wire x1="-4.826" y1="23.114" x2="-4.826" y2="27.94" width="0.1524" layer="91"/>
 <wire x1="-4.826" y1="27.94" x2="36.576" y2="27.94" width="0.1524" layer="91"/>
-<wire x1="39.116" y1="21.844" x2="36.576" y2="21.844" width="0.1524" layer="91"/>
+<wire x1="36.576" y1="18.034" x2="36.576" y2="21.844" width="0.1524" layer="91"/>
 <wire x1="36.576" y1="21.844" x2="36.576" y2="27.94" width="0.1524" layer="91"/>
+<wire x1="19.812" y1="18.034" x2="36.576" y2="18.034" width="0.1524" layer="91"/>
+<pinref part="U$5" gate="G$1" pin="1"/>
 <pinref part="U$5" gate="G$1" pin="4"/>
-<wire x1="17.272" y1="18.034" x2="36.576" y2="18.034" width="0.1524" layer="91"/>
-<wire x1="36.576" y1="18.034" x2="36.576" y2="21.844" width="0.1524" layer="91"/>
+<pinref part="IC1" gate="B" pin="+IN"/>
+<wire x1="38.862" y1="21.844" x2="36.576" y2="21.844" width="0.1524" layer="91"/>
 <junction x="36.576" y="21.844"/>
 </segment>
@@
 <net name="N$5" class="0">
 <segment>
-<pinref part="U$5" gate="G$1" pin="3"/>
-<wire x1="-3.048" y1="18.034" x2="-4.826" y2="18.034" width="0.1524" layer="91"/>
+<wire x1="-0.508" y1="18.034" x2="-4.826" y2="18.034" width="0.1524" layer="91"/>
 <wire x1="-4.826" y1="18.034" x2="-4.826" y2="11.684" width="0.1524" layer="91"/>
 <wire x1="-4.826" y1="11.684" x2="36.83" y2="11.684" width="0.1524" layer="91"/>
@@
 <pinref part="IC1" gate="B" pin="-IN"/>
 <wire x1="38.862" y1="16.764" x2="36.83" y2="16.764" width="0.1524" layer="91"/>
-<wire x1="17.526" y1="23.114" x2="18.034" y2="23.114" width="0.1524" layer="91"/>
-<wire x1="18.034" y1="23.114" x2="30.988" y2="23.114" width="0.1524" layer="91"/>
+<wire x1="17.526" y1="23.114" x2="19.812" y2="23.114" width="0.1524" layer="91"/>
+<wire x1="19.812" y1="23.114" x2="30.988" y2="23.114" width="0.1524" layer="91"/>
 <wire x1="30.988" y1="23.114" x2="30.988" y2="16.764" width="0.1524" layer="91"/>
 <wire x1="36.83" y1="16.764" x2="30.988" y2="16.764" width="0.1524" layer="91"/>
 <junction x="36.83" y="16.764"/>
+<wire x1="19.812" y1="23.114" x2="18.034" y2="23.114" width="0.1524" layer="91"/>
+<pinref part="U$5" gate="G$1" pin="3"/>
 <pinref part="U$5" gate="G$1" pin="6"/>
-<wire x1="17.272" y1="23.114" x2="17.526" y2="23.114" width="0.1524" layer="91"/>
+<junction x="19.812" y="23.114"/>
 </segment>
 </net>
@@
 <wire x1="28.702" y1="-6.604" x2="21.082" y2="-6.604" width="0.1524" layer="91"/>
 <wire x1="21.082" y1="-6.604" x2="21.082" y2="20.574" width="0.1524" layer="91"/>
+<wire x1="21.082" y1="20.574" x2="19.812" y2="20.574" width="0.1524" layer="91"/>
 <pinref part="U$5" gate="G$1" pin="5"/>
-<wire x1="21.082" y1="20.574" x2="17.272" y2="20.574" width="0.1524" layer="91"/>
 </segment>
 </net>
